Commit message: Added grippers to Wiktor.

File: wiktor_description/urdf/iiwa7.xacro (robot description, xacro)
@@ -289,16 +289,16 @@
             <parent link="${robot_name}_link_7"/>
             <child link="${robot_name}_link_ee"/>
-            <origin xyz="0 0 0.045" rpy="0 -${PI/2} 0"/>
+            <origin xyz="0 0 0.045" rpy="0 0 0"/>
         </joint>
         <link name="${robot_name}_link_ee">
         </link>
-        <joint name="${robot_name}_joint_ee_kuka" type="fixed">
-            <parent link="${robot_name}_link_7"/>
-            <child link="${robot_name}_link_ee_kuka"/>
-            <origin xyz="0 0 0.045" rpy="${PI} ${PI} ${PI}"/>
-            <axis xyz="0 0 1"/>
-        </joint>
-        <link name="${robot_name}_link_ee_kuka">
-        </link>
+        <!--<joint name="${robot_name}_joint_ee_kuka" type="fixed">-->
+            <!--<parent link="${robot_name}_link_7"/>-->
+            <!--<child link="${robot_name}_link_ee_kuka"/>-->
+            <!--<origin xyz="0 0 0.045" rpy="${PI} ${PI} ${PI}"/>-->
+            <!--<axis xyz="0 0 1"/>-->
+        <!--</joint>-->
+        <!--<link name="${robot_name}_link_ee_kuka">-->
+        <!--</link>-->
         <!--Extensions -->
         <xacro:iiwa_gazebo robot_name="${robot_name}"/>

File: wiktor_description/urdf/materials.xacro (robot description, xacro)
@@ -31,3 +31,6 @@
         <color rgba="0.2 0.2 0.2 1"/>
     </material>
+    <material name="DarkDarkGray">
+        <color rgba="0.1 0.1 0.1 1"/>
+    </material>
 </robot>

File: wiktor_description/urdf/wiktor.urdf (robot description, URDF)
Before this commit: robot wiktor, 26 links, 25 joints
Links:
- removed link wiktor_left_arm_link_ee_kuka
- removed link wiktor_right_arm_link_ee_kuka
- added link wiktor_left_gripper_fingerA_base, mass 1; collision mesh filename=package://wiktor_description/meshes/robotiq_3finger/finger_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; visual mesh filename=package://wiktor_description/meshes/robotiq_3finger/finger_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
- added link wiktor_left_gripper_fingerA_dist, mass 1; collision mesh filename=package://wiktor_description/meshes/robotiq_3finger/finger_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; visual mesh filename=package://wiktor_description/meshes/robotiq_3finger/finger_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
- added link wiktor_left_gripper_fingerA_med, mass 1; collision mesh filename=package://wiktor_description/meshes/robotiq_3finger/finger_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; visual mesh filename=package://wiktor_description/meshes/robotiq_3finger/finger_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
- added link wiktor_left_gripper_fingerA_prox, mass 1; collision mesh filename=package://wiktor_description/meshes/robotiq_3finger/finger_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; visual mesh filename=package://wiktor_description/meshes/robotiq_3finger/finger_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
- added link wiktor_left_gripper_fingerB_base, mass 1; collision mesh filename=package://wiktor_description/meshes/robotiq_3finger/finger_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; visual mesh filename=package://wiktor_description/meshes/robotiq_3finger/finger_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
- added link wiktor_left_gripper_fingerB_dist, mass 1; collision mesh filename=package://wiktor_description/meshes/robotiq_3finger/finger_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; visual mesh filename=package://wiktor_description/meshes/robotiq_3finger/finger_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
- added link wiktor_left_gripper_fingerB_med, mass 1; collision mesh filename=package://wiktor_description/meshes/robotiq_3finger/finger_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; visual mesh filename=package://wiktor_description/meshes/robotiq_3finger/finger_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
- added link wiktor_left_gripper_fingerB_prox, mass 1; collision mesh filename=package://wiktor_description/meshes/robotiq_3finger/finger_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; visual mesh filename=package://wiktor_description/meshes/robotiq_3finger/finger_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
- added link wiktor_left_gripper_fingerC_base, mass 1; collision mesh filename=package://wiktor_description/meshes/robotiq_3finger/finger_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; visual mesh filename=package://wiktor_description/meshes/robotiq_3finger/finger_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
- added link wiktor_left_gripper_fingerC_dist, mass 1; collision mesh filename=package://wiktor_description/meshes/robotiq_3finger/finger_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; visual mesh filename=package://wiktor_description/meshes/robotiq_3finger/finger_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
- added link wiktor_left_gripper_fingerC_med, mass 1; collision mesh filename=package://wiktor_description/meshes/robotiq_3finger/finger_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; visual mesh filename=package://wiktor_description/meshes/robotiq_3finger/finger_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
- added link wiktor_left_gripper_fingerC_prox, mass 1; collision mesh filename=package://wiktor_description/meshes/robotiq_3finger/finger_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; visual mesh filename=package://wiktor_description/meshes/robotiq_3finger/finger_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
- added link wiktor_left_gripper_mounting_bracket; collision mesh filename=package://wiktor_description/meshes/robotiq_3finger/kuka_to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; visual mesh filename=package://wiktor_description/meshes/robotiq_3finger/kuka_to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
- added link wiktor_left_gripper_palm, mass 1; collision mesh filename=package://wiktor_description/meshes/robotiq_3finger/palm_co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; visual mesh filename=package://wiktor_description/meshes/robotiq_3finger/palm_vi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
- added link wiktor_right_gripper_fingerA_base, mass 1; collision mesh filename=package://wiktor_description/meshes/robotiq_3finger/finger_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; visual mesh filename=package://wiktor_description/meshes/robotiq_3finger/finger_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
- added link wiktor_right_gripper_fingerA_dist, mass 1; collision mesh filename=package://wiktor_description/meshes/robotiq_3finger/finger_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; visual mesh filename=package://wiktor_description/meshes/robotiq_3finger/finger_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
- added link wiktor_right_gripper_fingerA_med, mass 1; collision mesh filename=package://wiktor_description/meshes/robotiq_3finger/finger_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; visual mesh filename=package://wiktor_description/meshes/robotiq_3finger/finger_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
- added link wiktor_right_gripper_fingerA_prox, mass 1; collision mesh filename=package://wiktor_description/meshes/robotiq_3finger/finger_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; visual mesh filename=package://wiktor_description/meshes/robotiq_3finger/finger_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
- added link wiktor_right_gripper_fingerB_base, mass 1; collision mesh filename=package://wiktor_description/meshes/robotiq_3finger/finger_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; visual mesh filename=package://wiktor_description/meshes/robotiq_3finger/finger_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
- added link wiktor_right_gripper_fingerB_dist, mass 1; collision mesh filename=package://wiktor_description/meshes/robotiq_3finger/finger_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; visual mesh filename=package://wiktor_description/meshes/robotiq_3finger/finger_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
- added link wiktor_right_gripper_fingerB_med, mass 1; collision mesh filename=package://wiktor_description/meshes/robotiq_3finger/finger_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; visual mesh filename=package://wiktor_description/meshes/robotiq_3finger/finger_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
- added link wiktor_right_gripper_fingerB_prox, mass 1; collision mesh filename=package://wiktor_description/meshes/robotiq_3finger/finger_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; visual mesh filename=package://wiktor_description/meshes/robotiq_3finger/finger_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
- added link wiktor_right_gripper_fingerC_base, mass 1; collision mesh filename=package://wiktor_description/meshes/robotiq_3finger/finger_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; visual mesh filename=package://wiktor_description/meshes/robotiq_3finger/finger_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
- added link wiktor_right_gripper_fingerC_dist, mass 1; collision mesh filename=package://wiktor_description/meshes/robotiq_3finger/finger_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; visual mesh filename=package://wiktor_description/meshes/robotiq_3finger/finger_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
- added link wiktor_right_gripper_fingerC_med, mass 1; collision mesh filename=package://wiktor_description/meshes/robotiq_3finger/finger_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; visual mesh filename=package://wiktor_description/meshes/robotiq_3finger/finger_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
- added link wiktor_right_gripper_fingerC_prox, mass 1; collision mesh filename=package://wiktor_description/meshes/robotiq_3finger/finger_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; visual mesh filename=package://wiktor_description/meshes/robotiq_3finger/finger_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
- added link wiktor_right_gripper_mounting_bracket; collision mesh filename=package://wiktor_description/meshes/robotiq_3finger/kuka_to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; visual mesh filename=package://wiktor_description/meshes/robotiq_3finger/kuka_to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
- added link wiktor_right_gripper_palm, mass 1; collision mesh filename=package://wiktor_description/meshes/robotiq_3finger/palm_co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; visual mesh filename=package://wiktor_description/meshes/robotiq_3finger/palm_vi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
Joints:
- removed joint wiktor_left_arm_joint_ee_kuka
- removed joint wiktor_right_arm_joint_ee_kuka
- added joint wiktor_left_arm_link_ee_wiktor_left_joint: type fixed, parent wiktor_left_arm_link_ee, child wiktor_left_gripper_mounting_bracket, origin xyz=0 0 0 rpy=0 0 0
- added joint wiktor_left_gripper_fingerA_joint_2: type revolute, parent wiktor_left_gripper_fingerA_base, child wiktor_left_gripper_fingerA_prox, origin xyz=0.02225000 0 0.02151380 rpy=0 0 0, axis 0 -1 0, limit lower=-1 upper=1 effort=300 velocity=10
- added joint wiktor_left_gripper_fingerA_joint_3: type revolute, parent wiktor_left_gripper_fingerA_prox, child wiktor_left_gripper_fingerA_med, origin xyz=0 0 0.05715000 rpy=0 0 0, axis 0 -1 0, limit lower=-1 upper=1 effort=300 velocity=10
- added joint wiktor_left_gripper_fingerA_joint_4: type revolute, parent wiktor_left_gripper_fingerA_med, child wiktor_left_gripper_fingerA_dist, origin xyz=0 0 0.03810000 rpy=0 0 0, axis 0 -1 0, limit lower=-1 upper=1 effort=300 velocity=10
- added joint wiktor_left_gripper_fingerA_knuckle: type fixed, parent wiktor_left_gripper_palm, child wiktor_left_gripper_fingerA_base, origin xyz=0.02225040 0 0.06111875 rpy=0 0 0
- added joint wiktor_left_gripper_fingerB_joint_2: type revolute, parent wiktor_left_gripper_fingerB_base, child wiktor_left_gripper_fingerB_prox, origin xyz=0.02225000 0 0.02151380 rpy=0 0 0, axis 0 -1 0, limit lower=-1 upper=1 effort=300 velocity=10
- added joint wiktor_left_gripper_fingerB_joint_3: type revolute, parent wiktor_left_gripper_fingerB_prox, child wiktor_left_gripper_fingerB_med, origin xyz=0 0 0.05715000 rpy=0 0 0, axis 0 -1 0, limit lower=-1 upper=1 effort=300 velocity=10
- added joint wiktor_left_gripper_fingerB_joint_4: type revolute, parent wiktor_left_gripper_fingerB_med, child wiktor_left_gripper_fingerB_dist, origin xyz=0 0 0.03810000 rpy=0 0 0, axis 0 -1 0, limit lower=-1 upper=1 effort=300 velocity=10
- added joint wiktor_left_gripper_fingerB_knuckle: type revolute, parent wiktor_left_gripper_palm, child wiktor_left_gripper_fingerB_base, origin xyz=-0.02230120 0.03651250 0.06111875 rpy=0 0 3.14159265359, axis -1 0 0, limit lower=-1 upper=1 effort=300 velocity=10
- added joint wiktor_left_gripper_fingerC_joint_2: type revolute, parent wiktor_left_gripper_fingerC_base, child wiktor_left_gripper_fingerC_prox, origin xyz=0.02225000 0 0.02151380 rpy=0 0 0, axis 0 -1 0, limit lower=-1 upper=1 effort=300 velocity=10
- added joint wiktor_left_gripper_fingerC_joint_3: type revolute, parent wiktor_left_gripper_fingerC_prox, child wiktor_left_gripper_fingerC_med, origin xyz=0 0 0.05715000 rpy=0 0 0, axis 0 -1 0, limit lower=-1 upper=1 effort=300 velocity=10
- added joint wiktor_left_gripper_fingerC_joint_4: type revolute, parent wiktor_left_gripper_fingerC_med, child wiktor_left_gripper_fingerC_dist, origin xyz=0 0 0.03810000 rpy=0 0 0, axis 0 -1 0, limit lower=-1 upper=1 effort=300 velocity=10
- added joint wiktor_left_gripper_fingerC_knuckle: type revolute, parent wiktor_left_gripper_palm, child wiktor_left_gripper_fingerC_base, origin xyz=-0.02230120 -0.03651250 0.06111875 rpy=0 0 3.14159265359, axis 1 0 0, limit lower=-1 upper=1 effort=300 velocity=10
- added joint wiktor_left_gripper_palm_joint: type fixed, parent wiktor_left_gripper_mounting_bracket, child wiktor_left_gripper_palm, origin xyz=0 0 0.02705 rpy=0 0 0.785398163397
- added joint wiktor_right_arm_link_ee_wiktor_right_joint: type fixed, parent wiktor_right_arm_link_ee, child wiktor_right_gripper_mounting_bracket, origin xyz=0 0 0 rpy=0 0 0
- added joint wiktor_right_gripper_fingerA_joint_2: type revolute, parent wiktor_right_gripper_fingerA_base, child wiktor_right_gripper_fingerA_prox, origin xyz=0.02225000 0 0.02151380 rpy=0 0 0, axis 0 -1 0, limit lower=-1 upper=1 effort=300 velocity=10
- added joint wiktor_right_gripper_fingerA_joint_3: type revolute, parent wiktor_right_gripper_fingerA_prox, child wiktor_right_gripper_fingerA_med, origin xyz=0 0 0.05715000 rpy=0 0 0, axis 0 -1 0, limit lower=-1 upper=1 effort=300 velocity=10
- added joint wiktor_right_gripper_fingerA_joint_4: type revolute, parent wiktor_right_gripper_fingerA_med, child wiktor_right_gripper_fingerA_dist, origin xyz=0 0 0.03810000 rpy=0 0 0, axis 0 -1 0, limit lower=-1 upper=1 effort=300 velocity=10
- added joint wiktor_right_gripper_fingerA_knuckle: type fixed, parent wiktor_right_gripper_palm, child wiktor_right_gripper_fingerA_base, origin xyz=0.02225040 0 0.06111875 rpy=0 0 0
- added joint wiktor_right_gripper_fingerB_joint_2: type revolute, parent wiktor_right_gripper_fingerB_base, child wiktor_right_gripper_fingerB_prox, origin xyz=0.02225000 0 0.02151380 rpy=0 0 0, axis 0 -1 0, limit lower=-1 upper=1 effort=300 velocity=10
- added joint wiktor_right_gripper_fingerB_joint_3: type revolute, parent wiktor_right_gripper_fingerB_prox, child wiktor_right_gripper_fingerB_med, origin xyz=0 0 0.05715000 rpy=0 0 0, axis 0 -1 0, limit lower=-1 upper=1 effort=300 velocity=10
- added joint wiktor_right_gripper_fingerB_joint_4: type revolute, parent wiktor_right_gripper_fingerB_med, child wiktor_right_gripper_fingerB_dist, origin xyz=0 0 0.03810000 rpy=0 0 0, axis 0 -1 0, limit lower=-1 upper=1 effort=300 velocity=10
- added joint wiktor_right_gripper_fingerB_knuckle: type revolute, parent wiktor_right_gripper_palm, child wiktor_right_gripper_fingerB_base, origin xyz=-0.02230120 0.03651250 0.06111875 rpy=0 0 3.14159265359, axis -1 0 0, limit lower=-1 upper=1 effort=300 velocity=10
- added joint wiktor_right_gripper_fingerC_joint_2: type revolute, parent wiktor_right_gripper_fingerC_base, child wiktor_right_gripper_fingerC_prox, origin xyz=0.02225000 0 0.02151380 rpy=0 0 0, axis 0 -1 0, limit lower=-1 upper=1 effort=300 velocity=10
- added joint wiktor_right_gripper_fingerC_joint_3: type revolute, parent wiktor_right_gripper_fingerC_prox, child wiktor_right_gripper_fingerC_med, origin xyz=0 0 0.05715000 rpy=0 0 0, axis 0 -1 0, limit lower=-1 upper=1 effort=300 velocity=10
- added joint wiktor_right_gripper_fingerC_joint_4: type revolute, parent wiktor_right_gripper_fingerC_med, child wiktor_right_gripper_fingerC_dist, origin xyz=0 0 0.03810000 rpy=0 0 0, axis 0 -1 0, limit lower=-1 upper=1 effort=300 velocity=10
- added joint wiktor_right_gripper_fingerC_knuckle: type revolute, parent wiktor_right_gripper_palm, child wiktor_right_gripper_fingerC_base, origin xyz=-0.02230120 -0.03651250 0.06111875 rpy=0 0 3.14159265359, axis 1 0 0, limit lower=-1 upper=1 effort=300 velocity=10
- added joint wiktor_right_gripper_palm_joint: type fixed, parent wiktor_right_gripper_mounting_bracket, child wiktor_right_gripper_palm, origin xyz=0 0 0.02705 rpy=0 0 0.785398163397
- joint wiktor_left_arm_joint_ee: origin xyz=0 0 0.045 rpy=0 -1.57079632679 0 -> xyz=0 0 0.045 rpy=0 0 0
- joint wiktor_right_arm_joint_ee: origin xyz=0 0 0.045 rpy=0 -1.57079632679 0 -> xyz=0 0 0.045 rpy=0 0 0

File: wiktor_description/urdf/wiktor.urdf.xacro (robot description, xacro)
@@ -20,3 +20,22 @@
         <origin xyz="0 0 0" rpy="0 0 0"/>
     </xacro:iiwa7>
+    <!-- arm to gripper adapter -->
+    <xacro:include filename="$(find wiktor_description)/urdf/iiwa7_to_robotiq_adapter.xacro"/>
+    <xacro:iia7_to_robotiq_adapter parent="$(arg robot_name)_left_arm_link_ee" prefix="$(arg robot_name)_left">
+        <!--<origin xyz="0 0 0" rpy="${PI/2} 0 ${PI/4}"/> &lt;!&ndash; Offset measured with a tape measure; please confirm/fix this value &ndash;&gt;-->
+        <origin xyz="0 0 0" rpy="0 0 0"/>
+    </xacro:iia7_to_robotiq_adapter>
+    <xacro:iia7_to_robotiq_adapter parent="$(arg robot_name)_right_arm_link_ee" prefix="$(arg robot_name)_right">
+        <!--<origin xyz="0 0 0" rpy="${PI/2} 0 ${PI/4}"/> &lt;!&ndash; Offset measured with a tape measure; please confirm/fix this value &ndash;&gt;-->
+        <origin xyz="0 0 0" rpy="0 0 0"/>
+    </xacro:iia7_to_robotiq_adapter>
+    <!-- Robotiq grippers -->
+    <!--Import the Robotiq 3 finger macro -->
+    <xacro:include filename="$(find wiktor_description)/urdf/robotiq_3finger_gripper.xacro"/>
+    <xacro:robotiq_3finger parent="$(arg robot_name)_left_gripper_mounting_bracket" prefix="$(arg robot_name)_left_gripper">
+        <origin xyz="0 0 0.02705" rpy="0 0 ${PI/4}"/> <!-- Offset measured with a tape measure; please confirm/fix this value -->
+    </xacro:robotiq_3finger>
+    <xacro:robotiq_3finger parent="$(arg robot_name)_right_gripper_mounting_bracket" prefix="$(arg robot_name)_right_gripper">
+        <origin xyz="0 0 0.02705" rpy="0 0 ${PI/4}"/> <!-- Offset measured with a tape measure; please confirm/fix this value -->
+    </xacro:robotiq_3finger>
 </robot>
