Commit message: fixed origins of joint angles for gripper

File: wiktor_description/urdf/robotiq_finger.xacro (robot description, xacro)
@@ -32,10 +32,10 @@
             <parent link="${prefix}_base"/>
             <child link="${prefix}_prox"/>
-            <origin xyz="0.02225000 0 0.02151380" rpy="0 0 0"/>
+            <origin xyz="0.02225000 0 0.02151380" rpy="0 ${35 * PI / 180} 0"/>
             <axis xyz="0 -1 0"/>
             <limit lower="-1" upper="1"
                    effort="${max_effort}" velocity="${max_velocity}"/>
-            <safety_controller soft_lower_limit="${-168 * PI / 180}"
-                               soft_upper_limit="${168 * PI / 180}"
+            <safety_controller soft_lower_limit="${-35 * PI / 180}"
+                               soft_upper_limit="${35 * PI / 180}"
                                k_position="${safety_controller_k_pos}"
                                k_velocity="${safety_controller_k_vel}"/>
@@ -102,5 +102,5 @@
             <parent link="${prefix}_med"/>
             <child link="${prefix}_dist"/>
-            <origin xyz="0 0 0.03810000" rpy="0 0 0"/>
+            <origin xyz="0 0 0.03810000" rpy="0 ${-23 * PI / 180} 0"/>
             <axis xyz="0 -1 0"/>
             <limit lower="-1" upper="1"

Commit message: bounds for finger joints

File: wiktor_description/urdf/robotiq_finger.xacro (robot description, xacro)
@@ -71,6 +71,6 @@
             <limit lower="-1" upper="1"
                    effort="${max_effort}" velocity="${max_velocity}"/>
-            <safety_controller soft_lower_limit="${-168 * PI / 180}"
-                               soft_upper_limit="${168 * PI / 180}"
+            <safety_controller soft_lower_limit="${0 * PI / 180}"
+                               soft_upper_limit="${90 * PI / 180}"
                                k_position="${safety_controller_k_pos}"
                                k_velocity="${safety_controller_k_vel}"/>
@@ -102,10 +102,10 @@
             <parent link="${prefix}_med"/>
             <child link="${prefix}_dist"/>
-            <origin xyz="0 0 0.03810000" rpy="0 ${-23 * PI / 180} 0"/>
+            <origin xyz="0 0 0.03810000" rpy="0 ${-25 * PI / 180} 0"/>
             <axis xyz="0 -1 0"/>
             <limit lower="-1" upper="1"
                    effort="${max_effort}" velocity="${max_velocity}"/>
-            <safety_controller soft_lower_limit="${-168 * PI / 180}"
-                               soft_upper_limit="${168 * PI / 180}"
+            <safety_controller soft_lower_limit="${-25 * PI / 180}"
+                               soft_upper_limit="${73 * PI / 180}"
                                k_position="${safety_controller_k_pos}"
                                k_velocity="${safety_controller_k_vel}"/>
