Commit message: Updated urdf file.

File: wiktor_description/urdf/iiwa7_to_robotiq_adapter.xacro (robot description, xacro)
@@ -24,67 +24,4 @@
             </collision>
         </link>
-        <!--<link name="${prefix}_iiwa_bracket">-->
-            <!--<visual>-->
-                <!--<origin xyz="0 0 0" rpy="0 0 0"/>-->
-                <!--<geometry>-->
-                    <!--<mesh filename="package://wiktor_description/meshes/robotiq_3finger/iiwa7_to_neutral_coupling_plate_visual.stl"/>-->
-                <!--</geometry>-->
-                <!--<material name="LightGrey"/>-->
-            <!--</visual>-->
-            <!--<collision>-->
-                <!--<origin xyz="0 0 0" rpy="0 0 0"/>-->
-                <!--<geometry>-->
-                    <!--<mesh filename="package://wiktor_description/meshes/robotiq_3finger/iiwa7_to_neutral_coupling_plate_collision.stl"/>-->
-                <!--</geometry>-->
-                <!--<material name="LightGrey"/>-->
-            <!--</collision>-->
-        <!--</link>-->
-        <!--<joint name="${prefix}_iiwa_to_robotiq_joint" type="fixed">-->
-            <!--<origin xyz="0 0 0.008" rpy="0 0 0"/>-->
-            <!--<parent link="${prefix}_iiwa_bracket"/>-->
-            <!--<child link="${prefix}_robotiq_bracket"/>-->
-        <!--</joint>-->
-        <!--<link name="${prefix}_robotiq_bracket">-->
-            <!--<visual>-->
-                <!--<origin xyz="0 0 0" rpy="0 0 0"/>-->
-                <!--<geometry>-->
-                    <!--<mesh filename="package://wiktor_description/meshes/robotiq_3finger/neutral_coupling_plate_to_robotiq_visual.stl"/>-->
-                <!--</geometry>-->
-                <!--<material name="DarkGrey"/>-->
-            <!--</visual>-->
-            <!--<collision>-->
-                <!--<origin xyz="0 0 0" rpy="0 0 0"/>-->
-                <!--<geometry>-->
-                    <!--<mesh filename="package://wiktor_description/meshes/robotiq_3finger/neutral_coupling_plate_to_robotiq_collision.stl"/>-->
-                <!--</geometry>-->
-                <!--<material name="DarkGrey"/>-->
-            <!--</collision>-->
-        <!--</link>-->
-        <!--<joint name="${prefix}_robotiq_gripper_mounting_bracket_joint" type="fixed">-->
-            <!--<origin xyz="0 0 0.1" rpy="0 0 0"/>-->
-            <!--<parent link="${prefix}_robotiq_bracket"/>-->
-            <!--<child link="${prefix}_gripper_mounting_bracket"/>-->
-        <!--</joint>-->
-        <!--<link name="${prefix}_gripper_mounting_bracket">-->
-            <!--<inertial>-->
-                <!--<origin xyz="0 0 0" rpy="0 0 0"/>-->
-                <!--<mass value="1"/>-->
-                <!--<inertia ixx="0.01" ixy="0" ixz="0" iyy="0.01" iyz="0" izz="0.01"/>-->
-            <!--</inertial>-->
-            <!--<visual>-->
-                <!--<origin xyz="0 0 0" rpy="0 0 0"/>-->
-                <!--<geometry>-->
-                    <!--<mesh filename="package://wiktor_description/meshes/robotiq_3finger/gripper_mounting_bracket_visual.stl"/>-->
-                <!--</geometry>-->
-                <!--<material name="DarkGray"/>-->
-            <!--</visual>-->
-            <!--<collision>-->
-                <!--<origin xyz="0 0 0" rpy="0 0 0"/>-->
-                <!--<geometry>-->
-                    <!--<mesh filename="package://wiktor_description/meshes/robotiq_3finger/gripper_mounting_bracket_collision.stl"/>-->
-                <!--</geometry>-->
-                <!--<material name="DarkGray"/>-->
-            <!--</collision>-->
-        <!--</link>-->
     </xacro:macro>
 </robot>

File: wiktor_description/urdf/wiktor.urdf (robot description, URDF)
Before this commit: robot wiktor, 52 links, 51 joints
Joints:
- joint wiktor_left_gripper_fingerA_joint_2: origin xyz=0.02225000 0 0.02151380 rpy=0 0 0 -> xyz=0.02225000 0 0.02151380 rpy=0 0.610865238198 0
- joint wiktor_left_gripper_fingerA_joint_4: origin xyz=0 0 0.03810000 rpy=0 0 0 -> xyz=0 0 0.03810000 rpy=0 -0.436332312999 0
- joint wiktor_left_gripper_fingerB_joint_2: origin xyz=0.02225000 0 0.02151380 rpy=0 0 0 -> xyz=0.02225000 0 0.02151380 rpy=0 0.610865238198 0
- joint wiktor_left_gripper_fingerB_joint_4: origin xyz=0 0 0.03810000 rpy=0 0 0 -> xyz=0 0 0.03810000 rpy=0 -0.436332312999 0
- joint wiktor_left_gripper_fingerC_joint_2: origin xyz=0.02225000 0 0.02151380 rpy=0 0 0 -> xyz=0.02225000 0 0.02151380 rpy=0 0.610865238198 0
- joint wiktor_left_gripper_fingerC_joint_4: origin xyz=0 0 0.03810000 rpy=0 0 0 -> xyz=0 0 0.03810000 rpy=0 -0.436332312999 0
- joint wiktor_right_gripper_fingerA_joint_2: origin xyz=0.02225000 0 0.02151380 rpy=0 0 0 -> xyz=0.02225000 0 0.02151380 rpy=0 0.610865238198 0
- joint wiktor_right_gripper_fingerA_joint_4: origin xyz=0 0 0.03810000 rpy=0 0 0 -> xyz=0 0 0.03810000 rpy=0 -0.436332312999 0
- joint wiktor_right_gripper_fingerB_joint_2: origin xyz=0.02225000 0 0.02151380 rpy=0 0 0 -> xyz=0.02225000 0 0.02151380 rpy=0 0.610865238198 0
- joint wiktor_right_gripper_fingerB_joint_4: origin xyz=0 0 0.03810000 rpy=0 0 0 -> xyz=0 0 0.03810000 rpy=0 -0.436332312999 0
- joint wiktor_right_gripper_fingerC_joint_2: origin xyz=0.02225000 0 0.02151380 rpy=0 0 0 -> xyz=0.02225000 0 0.02151380 rpy=0 0.610865238198 0
- joint wiktor_right_gripper_fingerC_joint_4: origin xyz=0 0 0.03810000 rpy=0 0 0 -> xyz=0 0 0.03810000 rpy=0 -0.436332312999 0
