Commit message: Added the palm surface link in the xacro

File: wiktor_description/urdf/robotiq_3finger_gripper.xacro (robot description, xacro)
@@ -28,4 +28,20 @@
                 <material name="DarkGray"/>
             </collision>
+        </link>
+        <!-- Palm surface aligned with the gripper axis -->
+        <joint name="${prefix}_palm_surface_joint" type="fixed">
+            <parent link="${prefix}_palm"/>
+            <child link="${prefix}_palm_surface"/>
+            <origin xyz="0 0 0.092075" rpy="0 0 0"/>
+        </joint>
+        <link name="${prefix}_palm_surface">
+        </link>
+        <!-- Palm surface aligned with the gripper axis -->
+        <joint name="${prefix}_palm_surface_kuka_joint" type="fixed">
+            <parent link="${prefix}_palm"/>
+            <child link="${prefix}_palm_surface_kuka"/>
+            <origin xyz="0 0 0.092075" rpy="0 0 -0.78539816339"/>
+        </joint>
+        <link name="${prefix}_palm_surface_kuka">
         </link>
         <!-- Finger A -->

File: wiktor_description/urdf/wiktor.urdf (robot description, URDF)
Before this commit: robot wiktor, 52 links, 51 joints
Links:
- added link wiktor_left_gripper_palm_surface
- added link wiktor_left_gripper_palm_surface_kuka
- added link wiktor_right_gripper_palm_surface
- added link wiktor_right_gripper_palm_surface_kuka
Joints:
- added joint wiktor_left_gripper_palm_surface_joint: type fixed, parent wiktor_left_gripper_palm, child wiktor_left_gripper_palm_surface, origin xyz=0 0 0.092075 rpy=0 0 0
- added joint wiktor_left_gripper_palm_surface_kuka_joint: type fixed, parent wiktor_left_gripper_palm, child wiktor_left_gripper_palm_surface_kuka, origin xyz=0 0 0.092075 rpy=0 0 -0.78539816339
- added joint wiktor_right_gripper_palm_surface_joint: type fixed, parent wiktor_right_gripper_palm, child wiktor_right_gripper_palm_surface, origin xyz=0 0 0.092075 rpy=0 0 0
- added joint wiktor_right_gripper_palm_surface_kuka_joint: type fixed, parent wiktor_right_gripper_palm, child wiktor_right_gripper_palm_surface_kuka, origin xyz=0 0 0.092075 rpy=0 0 -0.78539816339
