Commit message: Update the joint state publisher for the gripper, fix the urdf and xacro gripper model, change the scissor model joint limit

File: victor_description/urdf/robotiq_3finger_gripper.xacro (robot description, xacro)
@@ -58,8 +58,8 @@
             <child link="${prefix}_fingerB_base"/>
             <axis xyz="-1 0 0"/>
-            <limit lower="-1" upper="1"
+            <limit lower="${-16 * PI / 180}" upper="${10 * PI / 180}"
                effort="${max_effort}" velocity="${max_velocity}"/>
-            <safety_controller soft_lower_limit="${-168 * PI / 180}"
-                               soft_upper_limit="${168 * PI / 180}"
+            <safety_controller soft_lower_limit="${-14 * PI / 180}"
+                               soft_upper_limit="${8 * PI / 180}"
                                k_position="${safety_controller_k_pos}"
                                k_velocity="${safety_controller_k_vel}"/>
@@ -73,8 +73,8 @@
             <child link="${prefix}_fingerC_base"/>
             <axis xyz="1 0 0"/>
-            <limit lower="-1" upper="1"
+            <limit lower="${-16 * PI / 180}" upper="${10 * PI / 180}"
                effort="${max_effort}" velocity="${max_velocity}"/>
-            <safety_controller soft_lower_limit="${-168 * PI / 180}"
-                               soft_upper_limit="${168 * PI / 180}"
+            <safety_controller soft_lower_limit="${-14 * PI / 180}"
+                               soft_upper_limit="${8 * PI / 180}"
                                k_position="${safety_controller_k_pos}"
                                k_velocity="${safety_controller_k_vel}"/>

File: victor_description/urdf/victor.urdf (robot description, URDF)
Before this commit: robot victor, 56 links, 55 joints
Joints:
- joint victor_left_gripper_fingerB_knuckle: limit lower=-1 upper=1 effort=300 velocity=10 -> lower=-0.279252680319 upper=0.174532925199 effort=300 velocity=10
- joint victor_left_gripper_fingerC_knuckle: limit lower=-1 upper=1 effort=300 velocity=10 -> lower=-0.279252680319 upper=0.174532925199 effort=300 velocity=10
- joint victor_right_gripper_fingerB_knuckle: limit lower=-1 upper=1 effort=300 velocity=10 -> lower=-0.279252680319 upper=0.174532925199 effort=300 velocity=10
- joint victor_right_gripper_fingerC_knuckle: limit lower=-1 upper=1 effort=300 velocity=10 -> lower=-0.279252680319 upper=0.174532925199 effort=300 velocity=10
