Commit message: Updated joint limits for knuckle (joint 2) of each finger.

File: victor_description/urdf/robotiq_finger.xacro (robot description, xacro)
@@ -34,5 +34,5 @@
             <origin xyz="0.02225000 0 0.02151380" rpy="0 ${35 * PI / 180} 0"/>
             <axis xyz="0 -1 0"/>
-            <limit lower="-1" upper="1"
+            <limit lower="0" upper="1.2217304763960307"
                    effort="${max_effort}" velocity="${max_velocity}"/>
             <safety_controller soft_lower_limit="${-35 * PI / 180}"

File: victor_description/urdf/victor.urdf (robot description, URDF)
Before this commit: robot victor, 60 links, 59 joints
Joints:
- joint victor_left_gripper_fingerA_joint_2: limit lower=-1 upper=1 effort=300 velocity=10 -> lower=0 upper=1.2217304763960307 effort=300 velocity=10
- joint victor_left_gripper_fingerB_joint_2: limit lower=-1 upper=1 effort=300 velocity=10 -> lower=0 upper=1.2217304763960307 effort=300 velocity=10
- joint victor_left_gripper_fingerC_joint_2: limit lower=-1 upper=1 effort=300 velocity=10 -> lower=0 upper=1.2217304763960307 effort=300 velocity=10
- joint victor_right_gripper_fingerA_joint_2: limit lower=-1 upper=1 effort=300 velocity=10 -> lower=0 upper=1.2217304763960307 effort=300 velocity=10
- joint victor_right_gripper_fingerB_joint_2: limit lower=-1 upper=1 effort=300 velocity=10 -> lower=0 upper=1.2217304763960307 effort=300 velocity=10
- joint victor_right_gripper_fingerC_joint_2: limit lower=-1 upper=1 effort=300 velocity=10 -> lower=0 upper=1.2217304763960307 effort=300 velocity=10
