Commit message: changes to victor description

File: victor_description/urdf/iiwa.gazebo.xacro (robot description, xacro)
@@ -1,59 +1,53 @@
 <?xml version="1.0"?>
 <robot xmlns:xacro="http://www.ros.org/wiki/xacro">
-  <xacro:macro name="iiwa_gazebo" params="robot_name">
-    <!-- Load Gazebo lib and set the robot namespace -->
-    <gazebo>
-      <plugin name="gazebo_ros_control" filename="libgazebo_ros_control.so">
-        <robotNamespace>/${robot_name}</robotNamespace>
-      </plugin>
-    </gazebo>
-    <!-- Link0 -->
-    <gazebo reference="iiwa_link_0">
-      <material>Gazebo/Grey</material>
-      <mu1>0.2</mu1>
-      <mu2>0.2</mu2>
-    </gazebo>
-    <!-- Link1 -->
-    <gazebo reference="iiwa_link_1">
-      <material>Gazebo/Orange</material>
-      <mu1>0.2</mu1>
-      <mu2>0.2</mu2>
-    </gazebo>
-    <!-- Link2 -->
-    <gazebo reference="iiwa_link_2">
-      <material>Gazebo/Orange</material>
-      <mu1>0.2</mu1>
-      <mu2>0.2</mu2>
-    </gazebo>
-    <!-- Link3 -->
-    <gazebo reference="iiwa_link_3">
-      <material>Gazebo/Orange</material>
-      <mu1>0.2</mu1>
-      <mu2>0.2</mu2>
-    </gazebo>
-    <!-- Link4 -->
-    <gazebo reference="iiwa_link_4">
-      <material>Gazebo/Orange</material>
-      <mu1>0.2</mu1>
-      <mu2>0.2</mu2>
-    </gazebo>
-    <!-- Link5 -->
-    <gazebo reference="iiwa_link_5">
-      <material>Gazebo/Orange</material>
-      <mu1>0.2</mu1>
-      <mu2>0.2</mu2>
-    </gazebo>
-    <!-- Link6 -->
-    <gazebo reference="iiwa_link_6">
-      <material>Gazebo/Orange</material>
-      <mu1>0.2</mu1>
-      <mu2>0.2</mu2>
-    </gazebo>
-    <!-- Link7 -->
-    <gazebo reference="iiwa_link_7">
-      <material>Gazebo/Grey</material>
-      <mu1>0.2</mu1>
-      <mu2>0.2</mu2>
-    </gazebo>
-  </xacro:macro>
+    <xacro:macro name="iiwa_gazebo" params="robot_name kinematic">
+        <!-- Link0 -->
+        <gazebo reference="${robot_name}_link_0">
+            <kinematic>${kinematic}</kinematic>
+            <mu1>0.2</mu1>
+            <mu2>0.2</mu2>
+        </gazebo>
+        <!-- Link1 -->
+        <gazebo reference="${robot_name}_link_1">
+            <kinematic>${kinematic}</kinematic>
+            <mu1>0.2</mu1>
+            <mu2>0.2</mu2>
+        </gazebo>
+        <!-- Link2 -->
+        <gazebo reference="${robot_name}_link_2">
+            <kinematic>${kinematic}</kinematic>
+            <mu1>0.2</mu1>
+            <mu2>0.2</mu2>
+        </gazebo>
+        <!-- Link3 -->
+        <gazebo reference="${robot_name}_link_3">
+            <kinematic>${kinematic}</kinematic>
+            <mu1>0.2</mu1>
+            <mu2>0.2</mu2>
+        </gazebo>
+        <!-- Link4 -->
+        <gazebo reference="${robot_name}_link_4">
+            <kinematic>${kinematic}</kinematic>
+            <mu1>0.2</mu1>
+            <mu2>0.2</mu2>
+        </gazebo>
+        <!-- Link5 -->
+        <gazebo reference="${robot_name}_link_5">
+            <kinematic>${kinematic}</kinematic>
+            <mu1>0.2</mu1>
+            <mu2>0.2</mu2>
+        </gazebo>
+        <!-- Link6 -->
+        <gazebo reference="${robot_name}_link_6">
+            <kinematic>${kinematic}</kinematic>
+            <mu1>0.2</mu1>
+            <mu2>0.2</mu2>
+        </gazebo>
+        <!-- Link7 -->
+        <gazebo reference="${robot_name}_link_7">
+            <kinematic>${kinematic}</kinematic>
+            <mu1>0.2</mu1>
+            <mu2>0.2</mu2>
+        </gazebo>
+    </xacro:macro>
 </robot>

File: victor_description/urdf/iiwa7.xacro (robot description, xacro)
@@ -8,10 +8,8 @@
     <xacro:include filename="$(find victor_description)/urdf/utilities.xacro"/>
     <!-- some constants -->
-    <xacro:property name="safety_controller_k_pos" value="100"/>
-    <xacro:property name="safety_controller_k_vel" value="2"/>
     <xacro:property name="joint_damping" value="0.5"/>
     <xacro:property name="max_effort" value="300"/>
     <xacro:property name="max_velocity" value="10"/>
-    <xacro:macro name="iiwa7" params="parent hardware_interface robot_name *origin">
+    <xacro:macro name="iiwa7" params="parent hardware_interface robot_name kinematic *origin">
         <!--joint between {parent} and link_0-->
         <joint name="${parent}_${robot_name}_joint" type="fixed">
@@ -55,8 +53,4 @@
             <limit lower="${-170 * PI / 180}" upper="${170 * PI / 180}"
                    effort="${max_effort}" velocity="${max_velocity}"/>
-            <safety_controller soft_lower_limit="${-168 * PI / 180}"
-                               soft_upper_limit="${168 * PI / 180}"
-                               k_position="${safety_controller_k_pos}"
-                               k_velocity="${safety_controller_k_vel}"/>
             <dynamics damping="${joint_damping}"/>
         </joint>
@@ -89,8 +83,4 @@
             <limit lower="${-120 * PI / 180}" upper="${120 * PI / 180}"
                    effort="${max_effort}" velocity="${max_velocity}"/>
-            <safety_controller soft_lower_limit="${-118 * PI / 180}"
-                               soft_upper_limit="${118 * PI / 180}"
-                               k_position="${safety_controller_k_pos}"
-                               k_velocity="${safety_controller_k_vel}"/>
             <dynamics damping="${joint_damping}"/>
         </joint>
@@ -123,8 +113,4 @@
             <limit lower="${-170 * PI / 180}" upper="${170 * PI / 180}"
                    effort="${max_effort}" velocity="${max_velocity}"/>
-            <safety_controller soft_lower_limit="${-168 * PI / 180}"
-                               soft_upper_limit="${168 * PI / 180}"
-                               k_position="${safety_controller_k_pos}"
-                               k_velocity="${safety_controller_k_vel}"/>
             <dynamics damping="${joint_damping}"/>
         </joint>
@@ -157,8 +143,4 @@
             <limit lower="${-120 * PI / 180}" upper="${120 * PI / 180}"
                    effort="${max_effort}" velocity="${max_velocity}"/>
-            <safety_controller soft_lower_limit="${-118 * PI / 180}"
-                               soft_upper_limit="${118 * PI / 180}"
-                               k_position="${safety_controller_k_pos}"
-                               k_velocity="${safety_controller_k_vel}"/>
             <dynamics damping="${joint_damping}"/>
         </joint>
@@ -191,8 +173,4 @@
             <limit lower="${-170 * PI / 180}" upper="${170 * PI / 180}"
                    effort="${max_effort}" velocity="${max_velocity}"/>
-            <safety_controller soft_lower_limit="${-168 * PI / 180}"
-                               soft_upper_limit="${168 * PI / 180}"
-                               k_position="${safety_controller_k_pos}"
-                               k_velocity="${safety_controller_k_vel}"/>
             <dynamics damping="${joint_damping}"/>
         </joint>
@@ -225,8 +203,4 @@
             <limit lower="${-120 * PI / 180}" upper="${120 * PI / 180}"
                    effort="${max_effort}" velocity="${max_velocity}"/>
-            <safety_controller soft_lower_limit="${-118 * PI / 180}"
-                               soft_upper_limit="${118 * PI / 180}"
-                               k_position="${safety_controller_k_pos}"
-                               k_velocity="${safety_controller_k_vel}"/>
             <dynamics damping="${joint_damping}"/>
         </joint>
@@ -259,8 +233,4 @@
             <limit lower="${-175 * PI / 180}" upper="${175 * PI / 180}"
                    effort="${max_effort}" velocity="${max_velocity}"/>
-            <safety_controller soft_lower_limit="${-173 * PI / 180}"
-                               soft_upper_limit="${173 * PI / 180}"
-                               k_position="${safety_controller_k_pos}"
-                               k_velocity="${safety_controller_k_vel}"/>
             <dynamics damping="${joint_damping}"/>
         </joint>
@@ -302,6 +272,7 @@
         </link>
         <!--Extensions -->
-        <xacro:iiwa_gazebo robot_name="${robot_name}"/>
-        <xacro:iiwa_transmission hardware_interface="${hardware_interface}"/>
+        <xacro:iiwa_gazebo robot_name="${robot_name} ${kinematic}"/>
+        <xacro:iiwa_transmission hardware_interface="${hardware_interface}"
+                                 robot_name="${robot_name}"/>
     </xacro:macro>
 </robot>

File: victor_description/urdf/victor.urdf.xacro (robot description, xacro)
@@ -1,6 +1,8 @@
 <?xml version="1.0"?>
 <robot name="victor" xmlns:xacro="http://www.ros.org/wiki/xacro">
+    <xacro:property name="gripper" value="kinematic_robotiq" />
     <xacro:arg name="robot_name" default="victor"/>
-    <xacro:arg name="hardware_interface" default="PositionJointInterface"/>
+    <xacro:arg name="kinematic_arms" default="0"/>
+    <xacro:arg name="hardware_interface" default="hardware_interface/PositionJointInterface"/>
     <!-- Import Rviz colors -->
     <xacro:include filename="$(find victor_description)/urdf/materials.xacro"/>
@@ -15,5 +17,5 @@
     <xacro:include filename="$(find victor_description)/urdf/iiwa7.xacro"/>
     <xacro:iiwa7 hardware_interface="$(arg hardware_interface)" robot_name="$(arg robot_name)_left_arm"
-                 parent="$(arg robot_name)_left_arm_mount">
+                 parent="$(arg robot_name)_left_arm_mount" kinematic="$(arg kinematic_arms)">
         <origin xyz="0 0 0" rpy="0 0 0"/>
     </xacro:iiwa7>
@@ -26,5 +28,5 @@
     </link>
     <xacro:iiwa7 hardware_interface="$(arg hardware_interface)" robot_name="$(arg robot_name)_right_arm"
-                 parent="$(arg robot_name)_right_arm_mount">
+                 parent="$(arg robot_name)_right_arm_mount" kinematic="$(arg kinematic_arms)">
         <origin xyz="0 0 0" rpy="0 0 0"/>
     </xacro:iiwa7>
@@ -39,20 +41,26 @@
     <xacro:include filename="$(find victor_description)/urdf/iiwa7_to_robotiq_adapter.xacro"/>
     <xacro:iia7_to_robotiq_adapter parent="$(arg robot_name)_left_arm_flange" prefix="$(arg robot_name)_left">
-        <origin xyz="0 0 0" rpy="0 0 0"/>
+        <origin xyz="0 0 -0.01" rpy="0 0 0"/>
     </xacro:iia7_to_robotiq_adapter>
     <xacro:iia7_to_robotiq_adapter parent="$(arg robot_name)_right_arm_flange" prefix="$(arg robot_name)_right">
-        <origin xyz="0 0 0" rpy="0 0 0"/>
+        <origin xyz="0 0 -0.01" rpy="0 0 0"/>
     </xacro:iia7_to_robotiq_adapter>
     <!-- Robotiq grippers -->
-    <!--Import the Robotiq 3 finger macro -->
-    <xacro:include filename="$(find victor_description)/urdf/robotiq_3finger_gripper.xacro"/>
-    <xacro:robotiq_3finger parent="$(arg robot_name)_left_gripper_mounting_bracket" prefix="$(arg robot_name)_left_gripper">
-        <origin xyz="0 0 0.02705" rpy="0 0 ${PI/4}"/> <!-- Offset measured with a tape measure; please confirm/fix this value -->
-    </xacro:robotiq_3finger>
-    <xacro:robotiq_3finger parent="$(arg robot_name)_right_gripper_mounting_bracket" prefix="$(arg robot_name)_right_gripper">
-        <origin xyz="0 0 0.02705" rpy="0 0 ${PI/4}"/> <!-- Offset measured with a tape measure; please confirm/fix this value -->
-    </xacro:robotiq_3finger>
+    <xacro:if value="${gripper == 'kinematic_robotiq'}">
+        <xacro:include filename="$(find victor_description)/urdf/kinematic_robotiq_grippers.xacro"/>
+    </xacro:if>
+    <xacro:if value="${gripper == 'robotiq'}">
+        <xacro:include filename="$(find victor_description)/urdf/robotiq_grippers.xacro"/>
+    </xacro:if>
     <!-- Define additional links as "tools", which are useful for planning and getting transforms -->
     <xacro:include filename="$(find victor_description)/urdf/robotiq_pinch_grasp_tools.xacro"/>
     <xacro:robotiq_pinch_grasp_tools robot_name="$(arg robot_name)"/>
+    <!-- Add Gazebo properties for whole robot -->
+    <xacro:include filename="$(find victor_description)/urdf/victor.gazebo.xacro"/>
+    <xacro:include filename="$(find victor_description)/urdf/gazebo_utilities.xacro"/>
+    <!-- Load Gazebo lib and set the robot namespace -->
+    <xacro:add_gazebo_control_plugin robot_namespace="$(arg robot_name)"/>
+    <xacro:add_moveit_planning_scene_plugin robot_namespace="$(arg robot_name)" root_frame_id="victor_root"/>
+    <!-- Rigidly attach Victor to the Gazebo world -->
+    <xacro:add_gazebo_fixed_link base_link="$(arg robot_name)_root"/>
 </robot>
