Commit message: fix robot name param
tested with visualize_victor.launch

File: victor_description/urdf/robotiq_pinch_grasp_tools.xacro (robot description, xacro)
@@ -2,50 +2,52 @@
 <robot xmlns:xacro="http://www.ros.org/wiki/xacro">
     <xacro:arg name="tool_dist_to_link_7" default="0.254"/>
-    <link name="left_tool">
-        <visual name="left_tool_visual">
-            <origin xyz="0 0 0" rpy="0 0 0"/>
-            <geometry>
-                <sphere radius="0.002"/>
-            </geometry>
-        </visual>
-        <inertial>
-            <origin xyz="0 0 0" rpy="0 0 0"/>
-            <!-- It's important that these have non-zero mass, otherwise gazebos URDF to SDF conversion will ignore them -->
-            <mass value="0.00001"/>
-            <inertia ixx="0"
-                     ixy="0"
-                     ixz="0"
-                     iyy="0"
-                     iyz="0"
-                     izz="0"/>
-        </inertial>
-    </link>
-    <joint name="left_tool_joint" type="fixed">
-        <parent link="$(arg robot_name)_left_arm_link_7"/>
-        <child link="left_tool"/>
-        <origin xyz="0 0 $(arg tool_dist_to_link_7)"/>
-    </joint>
-    <link name="right_tool">
-        <visual name="right_tool_visual">
-            <origin xyz="0 0 0" rpy="0 0 0"/>
-            <geometry>
-                <sphere radius="0.002"/>
-            </geometry>
-        </visual>
-        <inertial>
-            <origin xyz="0 0 0" rpy="0 0 0"/>
-            <mass value="0.00001"/>
-            <inertia ixx="0"
-                     ixy="0"
-                     ixz="0"
-                     iyy="0"
-                     iyz="0"
-                     izz="0"/>
-        </inertial>
-    </link>
-    <joint name="right_tool_joint" type="fixed">
-        <parent link="$(arg robot_name)_right_arm_link_7"/>
-        <child link="right_tool"/>
-        <origin xyz="0 0 $(arg tool_dist_to_link_7)"/>
-    </joint>
+    <xacro:macro name="robotiq_pinch_grasp_tools" params="robot_name">
+        <link name="left_tool">
+            <visual name="left_tool_visual">
+                <origin xyz="0 0 0" rpy="0 0 0"/>
+                <geometry>
+                    <sphere radius="0.002"/>
+                </geometry>
+            </visual>
+            <inertial>
+                <origin xyz="0 0 0" rpy="0 0 0"/>
+                <!-- It's important that these have non-zero mass, otherwise gazebos URDF to SDF conversion will ignore them -->
+                <mass value="0.00001"/>
+                <inertia ixx="0"
+                         ixy="0"
+                         ixz="0"
+                         iyy="0"
+                         iyz="0"
+                         izz="0"/>
+            </inertial>
+        </link>
+        <joint name="left_tool_joint" type="fixed">
+            <parent link="$(arg robot_name)_left_arm_link_7"/>
+            <child link="left_tool"/>
+            <origin xyz="0 0 $(arg tool_dist_to_link_7)"/>
+        </joint>
+        <link name="right_tool">
+            <visual name="right_tool_visual">
+                <origin xyz="0 0 0" rpy="0 0 0"/>
+                <geometry>
+                    <sphere radius="0.002"/>
+                </geometry>
+            </visual>
+            <inertial>
+                <origin xyz="0 0 0" rpy="0 0 0"/>
+                <mass value="0.00001"/>
+                <inertia ixx="0"
+                         ixy="0"
+                         ixz="0"
+                         iyy="0"
+                         iyz="0"
+                         izz="0"/>
+            </inertial>
+        </link>
+        <joint name="right_tool_joint" type="fixed">
+            <parent link="$(arg robot_name)_right_arm_link_7"/>
+            <child link="right_tool"/>
+            <origin xyz="0 0 $(arg tool_dist_to_link_7)"/>
+        </joint>
+    </xacro:macro>
 </robot>

File: victor_description/urdf/victor.urdf.xacro (robot description, xacro)
@@ -55,3 +55,4 @@
     <!-- Define additional links as "tools", which are useful for planning and getting transforms -->
     <xacro:include filename="$(find victor_description)/urdf/robotiq_pinch_grasp_tools.xacro"/>
+    <xacro:robotiq_pinch_grasp_tools robot_name="$(arg robot_name)"/>
 </robot>

Commit message: mfaroni :

File: victor_description/urdf/robotiq_pinch_grasp_tools.xacro (robot description, xacro)
@@ -27,4 +27,28 @@
             <origin xyz="0 0 $(arg tool_dist_to_link_7)"/>
         </joint>
+        <link name="left_tool_2">
+            <visual name="left_tool_2_visual">
+                <origin xyz="0 0 0" rpy="0 0 0"/>
+                <geometry>
+                    <sphere radius="0.002"/>
+                </geometry>
+            </visual>
+            <inertial>
+                <origin xyz="0 0 0" rpy="0 0 0"/>
+                <!-- It's important that these have non-zero mass, otherwise gazebos URDF to SDF conversion will ignore them -->
+                <mass value="0.001"/>
+                <inertia ixx="0"
+                         ixy="0"
+                         ixz="0"
+                         iyy="0"
+                         iyz="0"
+                         izz="0"/>
+            </inertial>
+        </link>
+        <joint name="left_tool_2_joint" type="fixed">
+            <parent link="$(arg robot_name)_left_arm_link_7"/>
+            <child link="left_tool_2"/>
+            <origin xyz="0 0 $(arg tool_dist_to_link_7)" rpy="0 0 -0.785375"/>
+        </joint>
         <link name="right_tool">
             <visual name="right_tool_visual">
@@ -50,4 +74,27 @@
             <origin xyz="0 0 $(arg tool_dist_to_link_7)"/>
         </joint>
+        <link name="right_tool_2">
+            <visual name="right_tool_2_visual">
+                <origin xyz="0 0 0" rpy="0 0 0"/>
+                <geometry>
+                    <sphere radius="0.002"/>
+                </geometry>
+            </visual>
+            <inertial>
+                <origin xyz="0 0 0" rpy="0 0 0"/>
+                <mass value="0.001"/>
+                <inertia ixx="0"
+                         ixy="0"
+                         ixz="0"
+                         iyy="0"
+                         iyz="0"
+                         izz="0"/>
+            </inertial>
+        </link>
+        <joint name="right_tool_2_joint" type="fixed">
+            <parent link="$(arg robot_name)_right_arm_link_7"/>
+            <child link="right_tool_2"/>
+            <origin xyz="0 0 $(arg tool_dist_to_link_7)" rpy="0 0 -0.785375"/>
+        </joint>
     </xacro:macro>
 </robot>

File: victor_description/urdf/victor.urdf.xacro (robot description, xacro)
@@ -4,6 +4,6 @@
     <xacro:arg name="robot_name" default="victor"/>
     <xacro:arg name="kinematic_arms" default="0"/>
-    <!--<xacro:arg name="hardware_interface" default="hardware_interface/PositionJointInterface"/>-->
-    <xacro:arg name="hardware_interface" default="hardware_interface/EffortJointInterface"/>
+    <xacro:arg name="hardware_interface" default="hardware_interface/PositionJointInterface"/>
+    <!--<xacro:arg name="hardware_interface" default="hardware_interface/EffortJointInterface"/>-->
     <!-- Import Rviz colors -->
     <xacro:include filename="$(find victor_description)/urdf/materials.xacro"/>
