Commit message: change srdf to make more sense to me
rename tool frames to be robot generic

File: victor_description/urdf/victor.urdf.xacro (robot description, xacro)
@@ -53,4 +53,21 @@
         <origin xyz="0 0 0.02705" rpy="0 0 ${PI/4}"/> <!-- Offset measured with a tape measure; please confirm/fix this value -->
     </xacro:robotiq_3finger>
+    <!-- NOTE: defining tools here allows moveit to plan with respect to these frames very easily.
+      I think it makes sense to leave this file un-modified on shared accounts, and overwrite the robot description
+      on the parameter server from your local modified copy on a personal account. -->
+    <link name="left_tool_placeholder">
+    </link>
+    <joint name="$(arg robot_name)_left_tool_joint" type="fixed">
+        <parent link="$(arg robot_name)_left_gripper_palm_surface"/>
+        <child link="left_tool_placeholder"/>
+        <origin xyz="0 0 ${4 * 0.0254}"/>
+    </joint>
+    <link name="right_tool_placeholder">
+    </link>
+    <joint name="$(arg robot_name)_right_tool_joint" type="fixed">
+        <parent link="$(arg robot_name)_right_gripper_palm_surface"/>
+        <child link="right_tool_placeholder"/>
+        <origin xyz="0 0 ${4 * 0.0254}"/>
+    </joint>
     <!-- Add Gazebo properties for whole robot -->
     <xacro:include filename="$(find victor_description)/urdf/gazebo_utilities.xacro"/>

Commit message: preserve the tool links so the come through in gazebo

File: victor_description/urdf/victor.urdf.xacro (robot description, xacro)
@@ -61,16 +61,48 @@
       on the parameter server from your local modified copy on a personal account. -->
     <link name="left_tool_placeholder">
+        <visual name="left_tool_visual">
+            <origin xyz="0 0 0" rpy="0 0 0"/>
+            <geometry>
+                <sphere radius="0.002"/>
+            </geometry>
+        </visual>
+        <inertial>
+            <origin xyz="0 0 0" rpy="0 0 0"/>
+            <mass value="0.00001"/>
+            <inertia ixx="0"
+                     ixy="0"
+                     ixz="0"
+                     iyy="0"
+                     iyz="0"
+                     izz="0"/>
+        </inertial>
     </link>
-    <joint name="$(arg robot_name)_left_tool_joint" type="fixed">
-        <parent link="$(arg robot_name)_left_gripper_palm_surface"/>
+    <joint name="left_tool_joint" type="fixed">
+        <parent link="$(arg robot_name)_left_arm_link_7"/>
         <child link="left_tool_placeholder"/>
-        <origin xyz="0 0 ${4 * 0.0254}"/>
+        <origin xyz="0 0 ${10 * 0.0254}"/>
     </joint>
     <link name="right_tool_placeholder">
+        <visual name="right_tool_visual">
+            <origin xyz="0 0 0" rpy="0 0 0"/>
+            <geometry>
+                <sphere radius="0.002"/>
+            </geometry>
+        </visual>
+        <inertial>
+            <origin xyz="0 0 0" rpy="0 0 0"/>
+            <mass value="0.00001"/>
+            <inertia ixx="0"
+                     ixy="0"
+                     ixz="0"
+                     iyy="0"
+                     iyz="0"
+                     izz="0"/>
+        </inertial>
     </link>
-    <joint name="$(arg robot_name)_right_tool_joint" type="fixed">
-        <parent link="$(arg robot_name)_right_gripper_palm_surface"/>
+    <joint name="right_tool_joint" type="fixed">
+        <parent link="$(arg robot_name)_right_arm_link_7"/>
         <child link="right_tool_placeholder"/>
-        <origin xyz="0 0 ${4 * 0.0254}"/>
+        <origin xyz="0 0 ${10 * 0.0254}"/>
     </joint>
     <!-- Add Gazebo properties for whole robot -->

Commit message: add tool links

File: victor_description/urdf/victor.urdf.xacro (robot description, xacro)
@@ -1,7 +1,9 @@
 <?xml version="1.0"?>
 <robot name="victor" xmlns:xacro="http://www.ros.org/wiki/xacro">
+    <xacro:arg name="use_tools" default="true"/>
+    <xacro:arg name="tool_dist_to_link_7" default="0.254"/>
     <xacro:arg name="robot_name" default="victor"/>
     <xacro:arg name="hardware_interface" default="PositionJointInterface"/>
-        <!-- Import Rviz colors -->
+    <!-- Import Rviz colors -->
     <xacro:include filename="$(find victor_description)/urdf/materials.xacro"/>
     <!-- pedestal -->
@@ -14,5 +16,6 @@
     <!--Import the lbr iiwa macro -->
     <xacro:include filename="$(find victor_description)/urdf/iiwa7.xacro"/>
-    <xacro:iiwa7 hardware_interface="$(arg hardware_interface)" robot_name="$(arg robot_name)_left_arm" parent="$(arg robot_name)_left_arm_mount">
+    <xacro:iiwa7 hardware_interface="$(arg hardware_interface)" robot_name="$(arg robot_name)_left_arm"
+                 parent="$(arg robot_name)_left_arm_mount">
         <origin xyz="0 0 0" rpy="0 0 0"/>
     </xacro:iiwa7>
@@ -24,5 +27,6 @@
     <link name="$(arg robot_name)_left_arm_world_frame_kuka">
     </link>
-    <xacro:iiwa7 hardware_interface="$(arg hardware_interface)" robot_name="$(arg robot_name)_right_arm" parent="$(arg robot_name)_right_arm_mount">
+    <xacro:iiwa7 hardware_interface="$(arg hardware_interface)" robot_name="$(arg robot_name)_right_arm"
+                 parent="$(arg robot_name)_right_arm_mount">
         <origin xyz="0 0 0" rpy="0 0 0"/>
     </xacro:iiwa7>
@@ -37,11 +41,61 @@
     <xacro:include filename="$(find victor_description)/urdf/iiwa7_to_robotiq_adapter.xacro"/>
     <xacro:iia7_to_robotiq_adapter parent="$(arg robot_name)_left_arm_flange" prefix="$(arg robot_name)_left">
-        <!--<origin xyz="0 0 0" rpy="${PI/2} 0 ${PI/4}"/> &lt;!&ndash; Offset measured with a tape measure; please confirm/fix this value &ndash;&gt;-->
         <origin xyz="0 0 0" rpy="0 0 0"/>
     </xacro:iia7_to_robotiq_adapter>
     <xacro:iia7_to_robotiq_adapter parent="$(arg robot_name)_right_arm_flange" prefix="$(arg robot_name)_right">
-        <!--<origin xyz="0 0 0" rpy="${PI/2} 0 ${PI/4}"/> &lt;!&ndash; Offset measured with a tape measure; please confirm/fix this value &ndash;&gt;-->
         <origin xyz="0 0 0" rpy="0 0 0"/>
     </xacro:iia7_to_robotiq_adapter>
+    <xacro:if value="$(arg use_tools)">
+        <!-- NOTE: defining tools here allows moveit to plan with respect to these frames very easily.
+          I think it makes sense to leave this file un-modified on shared accounts, and overwrite the robot description
+          on the parameter server from your local modified copy on a personal account. -->
+        <link name="left_tool">
+            <visual name="left_tool_visual">
+                <origin xyz="0 0 0" rpy="0 0 0"/>
+                <geometry>
+                    <sphere radius="0.002"/>
+                </geometry>
+            </visual>
+            <inertial>
+                <origin xyz="0 0 0" rpy="0 0 0"/>
+                <!-- It's important that these have non-zero mass, otherwise gazebos URDF to SDF conversion will ignore them -->
+                <mass value="0.00001"/>
+                <inertia ixx="0"
+                         ixy="0"
+                         ixz="0"
+                         iyy="0"
+                         iyz="0"
+                         izz="0"/>
+            </inertial>
+        </link>
+        <joint name="left_tool_joint" type="fixed">
+            <parent link="$(arg robot_name)_left_arm_link_7"/>
+            <child link="left_tool"/>
+            <origin xyz="0 0 $(arg tool_dist_to_link_7)"/>
+        </joint>
+        <link name="right_tool">
+            <visual name="right_tool_visual">
+                <origin xyz="0 0 0" rpy="0 0 0"/>
+                <geometry>
+                    <sphere radius="0.002"/>
+                </geometry>
+            </visual>
+            <inertial>
+                <origin xyz="0 0 0" rpy="0 0 0"/>
+                <mass value="0.00001"/>
+                <inertia ixx="0"
+                         ixy="0"
+                         ixz="0"
+                         iyy="0"
+                         iyz="0"
+                         izz="0"/>
+            </inertial>
+        </link>
+        <joint name="right_tool_joint" type="fixed">
+            <parent link="$(arg robot_name)_right_arm_link_7"/>
+            <child link="right_tool"/>
+            <origin xyz="0 0 $(arg tool_dist_to_link_7)"/>
+        </joint>
+    </xacro:if>
     <!-- Robotiq grippers -->
     <!--Import the Robotiq 3 finger macro -->

Commit message: use separate tool files

File: victor_description/urdf/victor.urdf.xacro (robot description, xacro)
@@ -1,6 +1,4 @@
 <?xml version="1.0"?>
 <robot name="victor" xmlns:xacro="http://www.ros.org/wiki/xacro">
-    <xacro:arg name="use_tools" default="true"/>
-    <xacro:arg name="tool_dist_to_link_7" default="0.254"/>
     <xacro:arg name="robot_name" default="victor"/>
     <xacro:arg name="hardware_interface" default="PositionJointInterface"/>
@@ -46,56 +44,4 @@
         <origin xyz="0 0 0" rpy="0 0 0"/>
     </xacro:iia7_to_robotiq_adapter>
-    <xacro:if value="$(arg use_tools)">
-        <!-- NOTE: defining tools here allows moveit to plan with respect to these frames very easily.
-          I think it makes sense to leave this file un-modified on shared accounts, and overwrite the robot description
-          on the parameter server from your local modified copy on a personal account. -->
-        <link name="left_tool">
-            <visual name="left_tool_visual">
-                <origin xyz="0 0 0" rpy="0 0 0"/>
-                <geometry>
-                    <sphere radius="0.002"/>
-                </geometry>
-            </visual>
-            <inertial>
-                <origin xyz="0 0 0" rpy="0 0 0"/>
-                <!-- It's important that these have non-zero mass, otherwise gazebos URDF to SDF conversion will ignore them -->
-                <mass value="0.00001"/>
-                <inertia ixx="0"
-                         ixy="0"
-                         ixz="0"
-                         iyy="0"
-                         iyz="0"
-                         izz="0"/>
-            </inertial>
-        </link>
-        <joint name="left_tool_joint" type="fixed">
-            <parent link="$(arg robot_name)_left_arm_link_7"/>
-            <child link="left_tool"/>
-            <origin xyz="0 0 $(arg tool_dist_to_link_7)"/>
-        </joint>
-        <link name="right_tool">
-            <visual name="right_tool_visual">
-                <origin xyz="0 0 0" rpy="0 0 0"/>
-                <geometry>
-                    <sphere radius="0.002"/>
-                </geometry>
-            </visual>
-            <inertial>
-                <origin xyz="0 0 0" rpy="0 0 0"/>
-                <mass value="0.00001"/>
-                <inertia ixx="0"
-                         ixy="0"
-                         ixz="0"
-                         iyy="0"
-                         iyz="0"
-                         izz="0"/>
-            </inertial>
-        </link>
-        <joint name="right_tool_joint" type="fixed">
-            <parent link="$(arg robot_name)_right_arm_link_7"/>
-            <child link="right_tool"/>
-            <origin xyz="0 0 $(arg tool_dist_to_link_7)"/>
-        </joint>
-    </xacro:if>
     <!-- Robotiq grippers -->
     <!--Import the Robotiq 3 finger macro -->
@@ -107,3 +53,5 @@
         <origin xyz="0 0 0.02705" rpy="0 0 ${PI/4}"/> <!-- Offset measured with a tape measure; please confirm/fix this value -->
     </xacro:robotiq_3finger>
+    <!-- Define additional links as "tools", which are useful for planning and getting transforms -->
+    <xacro:include filename="$(find victor_description)/urdf/robotiq_pinch_grasp_tools.xacro"/>
 </robot>

Commit message: increase mass of fake tool links , somehow this fixes the overstretching issues

File: victor_description/urdf/victor.urdf.xacro (robot description, xacro)
@@ -69,5 +69,5 @@
         <inertial>
             <origin xyz="0 0 0" rpy="0 0 0"/>
-            <mass value="0.00001"/>
+            <mass value="0.01"/>
             <inertia ixx="0"
                      ixy="0"
@@ -92,5 +92,5 @@
         <inertial>
             <origin xyz="0 0 0" rpy="0 0 0"/>
-            <mass value="0.00001"/>
+            <mass value="0.01"/>
             <inertia ixx="0"
                      ixy="0"

Commit message: Preparation for gazebo testing with weight
- added attach/detach gazebo plugin
- took out grippers
- regenerated moveit_config
- added dirrt moveit planning pipeline

File: victor_description/urdf/victor.urdf.xacro (robot description, xacro)
@@ -1,8 +1,9 @@
 <?xml version="1.0"?>
 <robot name="victor" xmlns:xacro="http://www.ros.org/wiki/xacro">
-    <xacro:property name="gripper" value="kinematic_robotiq" />
+    <xacro:property name="gripper" value="none" />
     <xacro:arg name="robot_name" default="victor"/>
     <xacro:arg name="kinematic_arms" default="0"/>
     <xacro:arg name="hardware_interface" default="hardware_interface/PositionJointInterface"/>
+    <!--<xacro:arg name="hardware_interface" default="hardware_interface/EffortJointInterface"/> -->
     <!-- Import Rviz colors -->
     <xacro:include filename="$(find victor_description)/urdf/materials.xacro"/>

Commit message: added visual configuration for robotiq in gazebo and added services to simply open and close gripper

File: victor_description/urdf/victor.urdf.xacro (robot description, xacro)
@@ -1,5 +1,5 @@
 <?xml version="1.0"?>
 <robot name="victor" xmlns:xacro="http://www.ros.org/wiki/xacro">
-    <xacro:property name="gripper" value="none" />
+    <xacro:property name="gripper" value="visual_robotiq" />
     <xacro:arg name="robot_name" default="victor"/>
     <xacro:arg name="kinematic_arms" default="0"/>
@@ -54,4 +54,7 @@
         <xacro:include filename="$(find victor_description)/urdf/robotiq_grippers.xacro"/>
     </xacro:if>
+    <xacro:if value="${gripper == 'visual_robotiq'}">
+        <xacro:include filename="$(find victor_description)/urdf/robotiq_grippers_visual.xacro"/>
+    </xacro:if>
     <!-- Define additional links as "tools", which are useful for planning and getting transforms -->
     <xacro:include filename="$(find victor_description)/urdf/robotiq_pinch_grasp_tools.xacro"/>

Commit message: use new gripper models

File: victor_description/urdf/victor.urdf.xacro (robot description, xacro)
@@ -48,6 +48,19 @@
     <!-- Robotiq grippers -->
     <xacro:if value="${gripper == 'robotiq'}">
-        <xacro:include filename="$(find victor_description)/urdf/robotiq_grippers.xacro"/>
+        <xacro:include filename="$(find robotiq_3f_description)/urdf/robotiq_3f_gripper_macro.xacro"/>
+        <xacro:robotiq_3f_gripper prefix="$(arg robot_name)_left_" use_fake_hardware="false" usb_port="/dev/ttyUSB1"/>
+        <xacro:robotiq_3f_gripper prefix="$(arg robot_name)_right_" use_fake_hardware="false" usb_port="/dev/ttyUSB3"/>
+        <joint name="left_gripper_joint" type="fixed">
+            <parent link="$(arg robot_name)_left_gripper_mounting_bracket"/>
+            <child link="$(arg robot_name)_left_palm"/>
+            <origin xyz="0 0 0.0715" rpy="1.5707 0 0"/>
+        </joint>
+        <joint name="right_gripper_joint" type="fixed">
+            <parent link="$(arg robot_name)_right_gripper_mounting_bracket"/>
+            <child link="$(arg robot_name)_right_palm"/>
+            <origin xyz="0 0 0.0715" rpy="1.5707 0 0"/>
+        </joint>
     </xacro:if>
+    <!-- could have other grippers here for different values of "gripper"-->
     <!-- Define additional links as "tools", which are useful for planning and getting transforms -->
     <xacro:include filename="$(find victor_description)/urdf/robotiq_pinch_grasp_tools.xacro"/>
