Commit message: debugging launch file

File: victor_description/urdf/victor_torso.xacro (robot description, xacro)
@@ -19,5 +19,4 @@
                 <origin xyz="0 0 0.2" rpy="0 0 0"/>
                 <geometry>
-                    <!--<mesh filename="package://victor_description/meshes/torso_visual_model.stl"/>-->
                     <cylinder length="0.7" radius="0.2"/>
                 </geometry>
@@ -35,5 +34,4 @@
                 <origin xyz="0 0 -0.013" rpy="0 0 0"/>
                 <geometry>
-                    <!--<mesh filename="package://victor_description/meshes/torso_visual_model.stl"/>-->
                     <box size="0.31 0.31 0.032"/>
                 </geometry>
@@ -51,5 +49,4 @@
                 <origin xyz="0 0 -0.013" rpy="0 0 0"/>
                 <geometry>
-                    <!--<mesh filename="package://victor_description/meshes/torso_visual_model.stl"/>-->
                     <box size="0.31 0.31 0.032"/>
                 </geometry>
