Commit message: Added extra fixed joints and empty links directly into the URDF instead of as separate transform publishers.

File: victor_description/urdf/iiwa7.xacro (robot description, xacro)
@@ -286,19 +286,19 @@
             </collision>
         </link>
-        <joint name="${robot_name}_joint_ee" type="fixed">
+        <joint name="${robot_name}_joint_flange" type="fixed">
             <parent link="${robot_name}_link_7"/>
-            <child link="${robot_name}_link_ee"/>
+            <child link="${robot_name}_flange"/>
             <origin xyz="0 0 0.045" rpy="0 0 0"/>
         </joint>
-        <link name="${robot_name}_link_ee">
-        </link>
-        <!--<joint name="${robot_name}_joint_ee_kuka" type="fixed">-->
-            <!--<parent link="${robot_name}_link_7"/>-->
-            <!--<child link="${robot_name}_link_ee_kuka"/>-->
-            <!--<origin xyz="0 0 0.045" rpy="${PI} ${PI} ${PI}"/>-->
-            <!--<axis xyz="0 0 1"/>-->
-        <!--</joint>-->
-        <!--<link name="${robot_name}_link_ee_kuka">-->
-        <!--</link>-->
+        <link name="${robot_name}_flange">
+        </link>
+        <!-- Our usage above has been tweaked to match Kuka's internal usage, so identity transform -->
+        <joint name="${robot_name}_flange_kuka_joint" type="fixed">
+            <parent link="${robot_name}_flange"/>
+            <child link="${robot_name}_flange_kuka"/>
+            <origin xyz="0 0 0" rpy="0 0 0"/>
+        </joint>
+        <link name="${robot_name}_flange_kuka">
+        </link>
         <!--Extensions -->
         <xacro:iiwa_gazebo robot_name="${robot_name}"/>

File: victor_description/urdf/robotiq_3finger_gripper.xacro (robot description, xacro)
@@ -37,9 +37,9 @@
         <link name="${prefix}_palm_surface">
         </link>
-        <!-- Palm surface aligned with the gripper axis -->
+        <!-- Kuka internal frame has been changed to match our external usage, so identity transform -->
         <joint name="${prefix}_palm_surface_kuka_joint" type="fixed">
-            <parent link="${prefix}_palm"/>
+            <parent link="${prefix}_palm_surface"/>
             <child link="${prefix}_palm_surface_kuka"/>
-            <origin xyz="0 0 0.092075" rpy="0 0 -0.78539816339"/>
+            <origin xyz="0 0 0" rpy="0 0 0"/>
         </joint>
         <link name="${prefix}_palm_surface_kuka">

File: victor_description/urdf/victor.urdf (robot description, URDF)
Before this commit: robot victor, 56 links, 55 joints
Links:
- removed link victor_left_arm_link_ee
- removed link victor_right_arm_link_ee
- added link victor_left_arm_flange
- added link victor_left_arm_flange_kuka
- added link victor_left_arm_world_frame_kuka
- added link victor_right_arm_flange
- added link victor_right_arm_flange_kuka
- added link victor_right_arm_world_frame_kuka
Joints:
- removed joint victor_left_arm_joint_ee
- removed joint victor_left_arm_link_ee_victor_left_joint
- removed joint victor_right_arm_joint_ee
- removed joint victor_right_arm_link_ee_victor_right_joint
- added joint victor_joint_left_arm_world_frame_kuka: type fixed, parent victor_left_arm_mount, child victor_left_arm_world_frame_kuka, origin xyz=0 0 0 rpy=1.57079632679 0 0
- added joint victor_joint_right_arm_world_frame_kuka: type fixed, parent victor_right_arm_mount, child victor_right_arm_world_frame_kuka, origin xyz=0 0 0 rpy=-1.57079632679 0 0
- added joint victor_left_arm_flange_kuka_joint: type fixed, parent victor_left_arm_flange, child victor_left_arm_flange_kuka, origin xyz=0 0 0 rpy=0 0 0
- added joint victor_left_arm_flange_victor_left_joint: type fixed, parent victor_left_arm_flange, child victor_left_gripper_mounting_bracket, origin xyz=0 0 0 rpy=0 0 0
- added joint victor_left_arm_joint_flange: type fixed, parent victor_left_arm_link_7, child victor_left_arm_flange, origin xyz=0 0 0.045 rpy=0 0 0
- added joint victor_right_arm_flange_kuka_joint: type fixed, parent victor_right_arm_flange, child victor_right_arm_flange_kuka, origin xyz=0 0 0 rpy=0 0 0
- added joint victor_right_arm_flange_victor_right_joint: type fixed, parent victor_right_arm_flange, child victor_right_gripper_mounting_bracket, origin xyz=0 0 0 rpy=0 0 0
- added joint victor_right_arm_joint_flange: type fixed, parent victor_right_arm_link_7, child victor_right_arm_flange, origin xyz=0 0 0.045 rpy=0 0 0
- joint victor_left_gripper_palm_surface_kuka_joint: origin xyz=0 0 0.092075 rpy=0 0 -0.78539816339 -> xyz=0 0 0 rpy=0 0 0; parent victor_left_gripper_palm -> victor_left_gripper_palm_surface
- joint victor_right_gripper_palm_surface_kuka_joint: origin xyz=0 0 0.092075 rpy=0 0 -0.78539816339 -> xyz=0 0 0 rpy=0 0 0; parent victor_right_gripper_palm -> victor_right_gripper_palm_surface

File: victor_description/urdf/victor.urdf.xacro (robot description, xacro)
@@ -17,14 +17,28 @@
         <origin xyz="0 0 0" rpy="0 0 0"/>
     </xacro:iiwa7>
+    <joint name="$(arg robot_name)_joint_left_arm_world_frame_kuka" type="fixed">
+        <parent link="$(arg robot_name)_left_arm_mount"/>
+        <child link="$(arg robot_name)_left_arm_world_frame_kuka"/>
+        <origin xyz="0 0 0" rpy="1.57079632679 0 0"/>
+    </joint>
+    <link name="$(arg robot_name)_left_arm_world_frame_kuka">
+    </link>
     <xacro:iiwa7 hardware_interface="$(arg hardware_interface)" robot_name="$(arg robot_name)_right_arm" parent="$(arg robot_name)_right_arm_mount">
         <origin xyz="0 0 0" rpy="0 0 0"/>
     </xacro:iiwa7>
+    <joint name="$(arg robot_name)_joint_right_arm_world_frame_kuka" type="fixed">
+        <parent link="$(arg robot_name)_right_arm_mount"/>
+        <child link="$(arg robot_name)_right_arm_world_frame_kuka"/>
+        <origin xyz="0 0 0" rpy="-1.57079632679 0 0"/>
+    </joint>
+    <link name="$(arg robot_name)_right_arm_world_frame_kuka">
+    </link>
     <!-- arm to gripper adapter -->
     <xacro:include filename="$(find victor_description)/urdf/iiwa7_to_robotiq_adapter.xacro"/>
-    <xacro:iia7_to_robotiq_adapter parent="$(arg robot_name)_left_arm_link_ee" prefix="$(arg robot_name)_left">
+    <xacro:iia7_to_robotiq_adapter parent="$(arg robot_name)_left_arm_flange" prefix="$(arg robot_name)_left">
         <!--<origin xyz="0 0 0" rpy="${PI/2} 0 ${PI/4}"/> &lt;!&ndash; Offset measured with a tape measure; please confirm/fix this value &ndash;&gt;-->
         <origin xyz="0 0 0" rpy="0 0 0"/>
     </xacro:iia7_to_robotiq_adapter>
-    <xacro:iia7_to_robotiq_adapter parent="$(arg robot_name)_right_arm_link_ee" prefix="$(arg robot_name)_right">
+    <xacro:iia7_to_robotiq_adapter parent="$(arg robot_name)_right_arm_flange" prefix="$(arg robot_name)_right">
         <!--<origin xyz="0 0 0" rpy="${PI/2} 0 ${PI/4}"/> &lt;!&ndash; Offset measured with a tape measure; please confirm/fix this value &ndash;&gt;-->
         <origin xyz="0 0 0" rpy="0 0 0"/>

Commit message: set the max velocities in urdf to match joint_limits
this is important for gazebo simulation, because urdf joint speeds are
used by the gazebo ros joint controller

File: victor_description/urdf/iiwa7.xacro (robot description, xacro)
@@ -10,5 +10,4 @@
     <xacro:property name="joint_damping" value="0.5"/>
     <xacro:property name="max_effort" value="300"/>
-    <xacro:property name="max_velocity" value="10"/>
     <xacro:macro name="iiwa7" params="parent hardware_interface robot_name kinematic *origin">
         <!--joint between {parent} and link_0-->
@@ -52,5 +51,5 @@
             <axis xyz="0 0 1"/>
             <limit lower="${-170 * PI / 180}" upper="${170 * PI / 180}"
-                   effort="${max_effort}" velocity="${max_velocity}"/>
+                   effort="${max_effort}" velocity="1.7453292519943295"/>
             <dynamics damping="${joint_damping}"/>
         </joint>
@@ -82,5 +81,5 @@
             <axis xyz="0 0 1"/>
             <limit lower="${-120 * PI / 180}" upper="${120 * PI / 180}"
-                   effort="${max_effort}" velocity="${max_velocity}"/>
+                   effort="${max_effort}" velocity="1.7453292519943295"/>
             <dynamics damping="${joint_damping}"/>
         </joint>
@@ -112,5 +111,5 @@
             <axis xyz="0 0 1"/>
             <limit lower="${-170 * PI / 180}" upper="${170 * PI / 180}"
-                   effort="${max_effort}" velocity="${max_velocity}"/>
+                   effort="${max_effort}" velocity="1.7453292519943295"/>
             <dynamics damping="${joint_damping}"/>
         </joint>
@@ -142,5 +141,5 @@
             <axis xyz="0 0 1"/>
             <limit lower="${-120 * PI / 180}" upper="${120 * PI / 180}"
-                   effort="${max_effort}" velocity="${max_velocity}"/>
+                   effort="${max_effort}" velocity="2.2689280275926285"/>
             <dynamics damping="${joint_damping}"/>
         </joint>
@@ -172,5 +171,5 @@
             <axis xyz="0 0 1"/>
             <limit lower="${-170 * PI / 180}" upper="${170 * PI / 180}"
-                   effort="${max_effort}" velocity="${max_velocity}"/>
+                   effort="${max_effort}" velocity="2.443460952792061"/>
             <dynamics damping="${joint_damping}"/>
         </joint>
@@ -202,5 +201,5 @@
             <axis xyz="0 0 1"/>
             <limit lower="${-120 * PI / 180}" upper="${120 * PI / 180}"
-                   effort="${max_effort}" velocity="${max_velocity}"/>
+                   effort="${max_effort}" velocity="3.141592653589793"/>
             <dynamics damping="${joint_damping}"/>
         </joint>
@@ -232,5 +231,5 @@
             <axis xyz="0 0 1"/>
             <limit lower="${-175 * PI / 180}" upper="${175 * PI / 180}"
-                   effort="${max_effort}" velocity="${max_velocity}"/>
+                   effort="${max_effort}" velocity="3.141592653589793"/>
             <dynamics damping="${joint_damping}"/>
         </joint>

Commit message: delete gazebo stuff from robot description

File: victor_description/urdf/iiwa7.xacro (robot description, xacro)
@@ -1,8 +1,4 @@
 <?xml version="1.0"?>
 <robot xmlns:xacro="http://www.ros.org/wiki/xacro">
-    <!-- Import all Gazebo-customization elements, including Gazebo colors -->
-    <xacro:include filename="$(find victor_description)/urdf/iiwa.gazebo.xacro"/>
-    <!-- Import Transmissions -->
-    <xacro:include filename="$(find victor_description)/urdf/iiwa.transmission.xacro"/>
     <!-- Include Utilities -->
     <xacro:include filename="$(find victor_description)/urdf/utilities.xacro"/>
@@ -270,8 +266,4 @@
         <link name="${robot_name}_flange_kuka">
         </link>
-        <!--Extensions -->
-        <xacro:iiwa_gazebo robot_name="${robot_name}" kinematic="${kinematic}"/>
-        <xacro:iiwa_transmission hardware_interface="${hardware_interface}"
-                                 robot_name="${robot_name}"/>
     </xacro:macro>
 </robot>

File: victor_description/urdf/robotiq_pinch_grasp_tools.xacro (robot description, xacro)
@@ -12,5 +12,5 @@
             <inertial>
                 <origin xyz="0 0 0" rpy="0 0 0"/>
-                <!-- It's important that these have non-zero mass, otherwise gazebos URDF to SDF conversion will ignore them -->
+                <!-- These have non-zero mass, otherwise some URDF to SDF converters will ignore them -->
                 <mass value="0.001"/>
                 <inertia ixx="0"

File: victor_description/urdf/victor.urdf.xacro (robot description, xacro)
@@ -1,5 +1,5 @@
 <?xml version="1.0"?>
 <robot name="victor" xmlns:xacro="http://www.ros.org/wiki/xacro">
-    <xacro:property name="gripper" value="kinematic_robotiq" />
+    <xacro:property name="gripper" value="robotiq" />
     <xacro:arg name="robot_name" default="victor"/>
     <xacro:arg name="kinematic_arms" default="0"/>
@@ -47,7 +47,4 @@
     </xacro:iia7_to_robotiq_adapter>
     <!-- Robotiq grippers -->
-    <xacro:if value="${gripper == 'kinematic_robotiq'}">
-        <xacro:include filename="$(find victor_description)/urdf/kinematic_robotiq_grippers.xacro"/>
-    </xacro:if>
     <xacro:if value="${gripper == 'robotiq'}">
         <xacro:include filename="$(find victor_description)/urdf/robotiq_grippers.xacro"/>
@@ -56,11 +53,3 @@
     <xacro:include filename="$(find victor_description)/urdf/robotiq_pinch_grasp_tools.xacro"/>
     <xacro:robotiq_pinch_grasp_tools robot_name="$(arg robot_name)"/>
-    <!-- Add Gazebo properties for whole robot -->
-    <xacro:include filename="$(find victor_description)/urdf/victor.gazebo.xacro"/>
-    <xacro:include filename="$(find victor_description)/urdf/gazebo_utilities.xacro"/>
-    <!-- Load Gazebo lib and set the robot namespace -->
-    <xacro:add_gazebo_control_plugin robot_namespace="$(arg robot_name)"/>
-    <xacro:add_moveit_planning_scene_plugin robot_namespace="$(arg robot_name)" root_frame_id="victor_root"/>
-    <!-- Rigidly attach Victor to the Gazebo world -->
-    <xacro:add_gazebo_fixed_link base_link="$(arg robot_name)_root"/>
 </robot>

Commit message: fix the wrench frame and still have a problem on mismatch time for kuka control machine

File: victor_description/urdf/iiwa7.xacro (robot description, xacro)
@@ -258,11 +258,11 @@
         <link name="${robot_name}_flange">
         </link>
-        <!-- Our usage above has been tweaked to match Kuka's internal usage, so identity transform -->
+        <!-- This is the frame in which the external wrench is computer by the Kuka Java code (Sunrise). -->
         <joint name="${robot_name}_flange_kuka_joint" type="fixed">
             <parent link="${robot_name}_flange"/>
-            <child link="${robot_name}_flange_kuka"/>
-            <origin xyz="0 0 0" rpy="0 0 0"/>
-        </joint>
-        <link name="${robot_name}_flange_kuka">
+            <child link="${robot_name}_sunrise_palm_surface"/>
+            <origin xyz="0 0 0.119" rpy="0 0 0.78539"/>
+        </joint>
+        <link name="${robot_name}_sunrise_palm_surface">
         </link>
     </xacro:macro>

File: victor_description/urdf/victor.urdf.xacro (robot description, xacro)
@@ -54,15 +54,11 @@
             <parent link="$(arg robot_name)_left_gripper_mounting_bracket"/>
             <child link="$(arg robot_name)_left_palm"/>
-            <origin xyz="0 0 0.0715" rpy="1.5707 0 0"/>
+            <origin xyz="0 0 0.0715" rpy="1.5707 0 0.78539"/>
         </joint>
         <joint name="right_gripper_joint" type="fixed">
             <parent link="$(arg robot_name)_right_gripper_mounting_bracket"/>
             <child link="$(arg robot_name)_right_palm"/>
-            <origin xyz="0 0 0.0715" rpy="1.5707 0 0"/>
+            <origin xyz="0 0 0.0715" rpy="1.5707 0 0.78539"/>
         </joint>
     </xacro:if>
-    <!-- could have other grippers here for different values of "gripper"-->
-    <!-- Define additional links as "tools", which are useful for planning and getting transforms -->
-    <xacro:include filename="$(find victor_description)/urdf/robotiq_pinch_grasp_tools.xacro"/>
-    <xacro:robotiq_pinch_grasp_tools robot_name="$(arg robot_name)"/>
 </robot>

Commit message: tweak params and add frame for cartesian commands to urdf

File: victor_description/urdf/iiwa7.xacro (robot description, xacro)
@@ -40,4 +40,12 @@
             </self_collision_checking>
         </link>
+        <!--joint and link for cartesian commands -->
+        <joint name="${robot_name}_cartesian_cmd_joint" type="fixed">
+            <origin xyz="0 0 0" rpy="${PI/2} 0 0"/>
+            <parent link="${robot_name}_link_0"/>
+            <child link="${robot_name}_cartesian_cmd"/>
+        </joint>
+        <link name="${robot_name}_cartesian_cmd">
+        </link>
         <!-- joint between link_0 and link_1 -->
         <joint name="${robot_name}_joint_1" type="revolute">

Commit message: fix right arm cartesian cmd base frame

File: victor_description/urdf/iiwa7.xacro (robot description, xacro)
@@ -40,12 +40,4 @@
             </self_collision_checking>
         </link>
-        <!--joint and link for cartesian commands -->
-        <joint name="${robot_name}_cartesian_cmd_joint" type="fixed">
-            <origin xyz="0 0 0" rpy="${PI/2} 0 0"/>
-            <parent link="${robot_name}_link_0"/>
-            <child link="${robot_name}_cartesian_cmd"/>
-        </joint>
-        <link name="${robot_name}_cartesian_cmd">
-        </link>
         <!-- joint between link_0 and link_1 -->
         <joint name="${robot_name}_joint_1" type="revolute">

File: victor_description/urdf/victor.urdf.xacro (robot description, xacro)
@@ -46,4 +46,19 @@
         <origin xyz="0 0 -0.01" rpy="0 0 0"/>
     </xacro:iia7_to_robotiq_adapter>
+    <!-- Cartesian commands -->
+    <joint name="$(arg robot_name)_left_arm_cartesian_cmd_joint" type="fixed">
+        <origin xyz="0 0 0" rpy="${PI/2} 0 0"/>
+        <parent link="$(arg robot_name)_left_arm_link_0"/>
+        <child link="$(arg robot_name)_left_arm_cartesian_cmd"/>
+    </joint>
+    <link name="$(arg robot_name)_left_arm_cartesian_cmd">
+    </link>
+    <joint name="$(arg robot_name)_right_arm_cartesian_cmd_joint" type="fixed">
+        <origin xyz="0 0 0" rpy="-${PI/2} 0 0"/>
+        <parent link="$(arg robot_name)_right_arm_link_0"/>
+        <child link="$(arg robot_name)_right_arm_cartesian_cmd"/>
+    </joint>
+    <link name="$(arg robot_name)_right_arm_cartesian_cmd">
+    </link>
     <!-- Robotiq grippers -->
     <xacro:if value="${gripper == 'robotiq'}">

Commit message: cable routing done

File: victor_description/urdf/iiwa7.xacro (robot description, xacro)
@@ -136,5 +136,5 @@
             <origin xyz="0 0 0.19" rpy="${PI / 2} 0 0"/>
             <axis xyz="0 0 1"/>
-            <limit lower="${-120 * PI / 180}" upper="${120 * PI / 180}"
+            <limit lower="${-120 * PI / 180}" upper="${119 * PI / 180}"
                    effort="${max_effort}" velocity="2.2689280275926285"/>
             <dynamics damping="${joint_damping}"/>

Commit message: change robot config

File: victor_description/urdf/iiwa7.xacro (robot description, xacro)
@@ -76,5 +76,5 @@
             <origin xyz="0 0 0.19" rpy="${PI / 2}   0 ${PI}"/>
             <axis xyz="0 0 1"/>
-            <limit lower="${-120 * PI / 180}" upper="${119 * PI / 180}"
+            <limit lower="${-119 * PI / 180}" upper="${119 * PI / 180}"
                    effort="${max_effort}" velocity="1.7453292519943295"/>
             <dynamics damping="${joint_damping}"/>
@@ -106,5 +106,5 @@
             <origin xyz="0 0.21 0" rpy="${PI / 2} 0 ${PI}"/>
             <axis xyz="0 0 1"/>
-            <limit lower="${-170 * PI / 180}" upper="${170 * PI / 180}"
+            <limit lower="${-169 * PI / 180}" upper="${169 * PI / 180}"
                    effort="${max_effort}" velocity="1.7453292519943295"/>
             <dynamics damping="${joint_damping}"/>
@@ -136,5 +136,5 @@
             <origin xyz="0 0 0.19" rpy="${PI / 2} 0 0"/>
             <axis xyz="0 0 1"/>
-            <limit lower="${-120 * PI / 180}" upper="${119 * PI / 180}"
+            <limit lower="${-119 * PI / 180}" upper="${119 * PI / 180}"
                    effort="${max_effort}" velocity="2.2689280275926285"/>
             <dynamics damping="${joint_damping}"/>
@@ -166,5 +166,5 @@
             <origin xyz="0 0.21 0" rpy="${-PI / 2} ${PI} 0"/>
             <axis xyz="0 0 1"/>
-            <limit lower="${-170 * PI / 180}" upper="${170 * PI / 180}"
+            <limit lower="${-169 * PI / 180}" upper="${169 * PI / 180}"
                    effort="${max_effort}" velocity="2.443460952792061"/>
             <dynamics damping="${joint_damping}"/>
@@ -196,5 +196,5 @@
             <origin xyz="0 0.06070 0.19" rpy="${PI / 2} 0 0"/>
             <axis xyz="0 0 1"/>
-            <limit lower="${-120 * PI / 180}" upper="${120 * PI / 180}"
+            <limit lower="${-119 * PI / 180}" upper="${119 * PI / 180}"
                    effort="${max_effort}" velocity="3.141592653589793"/>
             <dynamics damping="${joint_damping}"/>
