Commit message: Added victor with adapter

File: victor_description/urdf/iiwa7_to_robotiq_adapter.xacro (robot description, xacro)
@@ -1,5 +1,5 @@
 <?xml version="1.0"?>
 <robot xmlns:xacro="http://www.ros.org/wiki/xacro">
-    <xacro:macro name="iia7_to_robotiq_adapter" params="parent prefix *origin">
+    <xacro:macro name="iiwa7_to_robotiq_adapter" params="parent prefix *origin">
         <!--joint between {parent} and link_0-->
         <joint name="${parent}_${prefix}_joint" type="fixed">

File: victor_description/urdf/victor.urdf.xacro (robot description, xacro)
@@ -55,10 +55,10 @@
     <!-- arm to gripper adapter -->
     <xacro:include filename="$(find victor_description)/urdf/iiwa7_to_robotiq_adapter.xacro"/>
-    <xacro:iia7_to_robotiq_adapter parent="$(arg robot_name)_left_arm_flange" prefix="$(arg robot_name)_left">
+    <xacro:iiwa7_to_robotiq_adapter parent="$(arg robot_name)_left_arm_flange" prefix="$(arg robot_name)_left">
         <origin xyz="0 0 -0.01" rpy="0 0 0"/>
-    </xacro:iia7_to_robotiq_adapter>
-    <xacro:iia7_to_robotiq_adapter parent="$(arg robot_name)_right_arm_flange" prefix="$(arg robot_name)_right">
+    </xacro:iiwa7_to_robotiq_adapter>
+    <xacro:iiwa7_to_robotiq_adapter parent="$(arg robot_name)_right_arm_flange" prefix="$(arg robot_name)_right">
         <origin xyz="0 0 -0.01" rpy="0 0 0"/>
-    </xacro:iia7_to_robotiq_adapter>
+    </xacro:iiwa7_to_robotiq_adapter>
     <!-- Robotiq grippers -->
     <xacro:if value="${gripper == 'robotiq'}">
