Commit message: take out gripper from srdf

File: victor_moveit_config/config/gazebo_victor.urdf (robot description, URDF)
Before this commit: robot victor, 59 links, 58 joints
Links:
- removed link l_finger_1_link_0
- removed link l_finger_1_link_1
- removed link l_finger_1_link_2
- removed link l_finger_1_link_3
- removed link l_finger_2_link_0
- removed link l_finger_2_link_1
- removed link l_finger_2_link_2
- removed link l_finger_2_link_3
- removed link l_finger_middle_link_0
- removed link l_finger_middle_link_1
- removed link l_finger_middle_link_2
- removed link l_finger_middle_link_3
- removed link l_palm
- removed link r_finger_1_link_0
- removed link r_finger_1_link_1
- removed link r_finger_1_link_2
- removed link r_finger_1_link_3
- removed link r_finger_2_link_0
- removed link r_finger_2_link_1
- removed link r_finger_2_link_2
- removed link r_finger_2_link_3
- removed link r_finger_middle_link_0
- removed link r_finger_middle_link_1
- removed link r_finger_middle_link_2
- removed link r_finger_middle_link_3
- removed link r_palm
Joints:
- removed joint l_finger_1_joint_1
- removed joint l_finger_1_joint_2
- removed joint l_finger_1_joint_3
- removed joint l_finger_2_joint_1
- removed joint l_finger_2_joint_2
- removed joint l_finger_2_joint_3
- removed joint l_finger_middle_joint_1
- removed joint l_finger_middle_joint_2
- removed joint l_finger_middle_joint_3
- removed joint l_palm_finger_1_joint
- removed joint l_palm_finger_2_joint
- removed joint l_palm_finger_middle_joint
- removed joint l_robotiq_hand_joint
- removed joint r_finger_1_joint_1
- removed joint r_finger_1_joint_2
- removed joint r_finger_1_joint_3
- removed joint r_finger_2_joint_1
- removed joint r_finger_2_joint_2
- removed joint r_finger_2_joint_3
- removed joint r_finger_middle_joint_1
- removed joint r_finger_middle_joint_2
- removed joint r_finger_middle_joint_3
- removed joint r_palm_finger_1_joint
- removed joint r_palm_finger_2_joint
- removed joint r_palm_finger_middle_joint
- removed joint r_robotiq_hand_joint
