Commit message: add fingers to HW iface

File: victor_moveit_config/config/victor.ros2_control.xacro (robot description, xacro)
@@ -19,5 +19,4 @@
                   <param name="initial_value">${initial_positions['victor_left_arm_joint_1']}</param>
                 </state_interface>
-                <state_interface name="velocity"/>
                 <state_interface name="effort"/>
                 <state_interface name="external_torque"/>
@@ -28,5 +27,4 @@
                   <param name="initial_value">${initial_positions['victor_left_arm_joint_2']}</param>
                 </state_interface>
-                <state_interface name="velocity"/>
                 <state_interface name="effort"/>
                 <state_interface name="external_torque"/>
@@ -37,5 +35,4 @@
                   <param name="initial_value">${initial_positions['victor_left_arm_joint_3']}</param>
                 </state_interface>
-                <state_interface name="velocity"/>
                 <state_interface name="effort"/>
                 <state_interface name="external_torque"/>
@@ -46,5 +43,4 @@
                   <param name="initial_value">${initial_positions['victor_left_arm_joint_4']}</param>
                 </state_interface>
-                <state_interface name="velocity"/>
                 <state_interface name="effort"/>
                 <state_interface name="external_torque"/>
@@ -55,5 +51,4 @@
                   <param name="initial_value">${initial_positions['victor_left_arm_joint_5']}</param>
                 </state_interface>
-                <state_interface name="velocity"/>
                 <state_interface name="effort"/>
                 <state_interface name="external_torque"/>
@@ -64,5 +59,4 @@
                   <param name="initial_value">${initial_positions['victor_left_arm_joint_6']}</param>
                 </state_interface>
-                <state_interface name="velocity"/>
                 <state_interface name="effort"/>
                 <state_interface name="external_torque"/>
@@ -73,5 +67,4 @@
                   <param name="initial_value">${initial_positions['victor_left_arm_joint_7']}</param>
                 </state_interface>
-                <state_interface name="velocity"/>
                 <state_interface name="effort"/>
                 <state_interface name="external_torque"/>
@@ -82,5 +75,4 @@
                   <param name="initial_value">${initial_positions['victor_right_arm_joint_1']}</param>
                 </state_interface>
-                <state_interface name="velocity"/>
                 <state_interface name="effort"/>
                 <state_interface name="external_torque"/>
@@ -91,5 +83,4 @@
                   <param name="initial_value">${initial_positions['victor_right_arm_joint_2']}</param>
                 </state_interface>
-                <state_interface name="velocity"/>
                 <state_interface name="effort"/>
                 <state_interface name="external_torque"/>
@@ -100,5 +91,4 @@
                   <param name="initial_value">${initial_positions['victor_right_arm_joint_3']}</param>
                 </state_interface>
-                <state_interface name="velocity"/>
                 <state_interface name="effort"/>
                 <state_interface name="external_torque"/>
@@ -109,5 +99,4 @@
                   <param name="initial_value">${initial_positions['victor_right_arm_joint_4']}</param>
                 </state_interface>
-                <state_interface name="velocity"/>
                 <state_interface name="effort"/>
                 <state_interface name="external_torque"/>
@@ -118,5 +107,4 @@
                   <param name="initial_value">${initial_positions['victor_right_arm_joint_5']}</param>
                 </state_interface>
-                <state_interface name="velocity"/>
                 <state_interface name="effort"/>
                 <state_interface name="external_torque"/>
@@ -127,5 +115,4 @@
                   <param name="initial_value">${initial_positions['victor_right_arm_joint_6']}</param>
                 </state_interface>
-                <state_interface name="velocity"/>
                 <state_interface name="effort"/>
                 <state_interface name="external_torque"/>
@@ -136,7 +123,10 @@
                   <param name="initial_value">${initial_positions['victor_right_arm_joint_7']}</param>
                 </state_interface>
-                <state_interface name="velocity"/>
                 <state_interface name="effort"/>
                 <state_interface name="external_torque"/>
+            </joint>
+            <joint name="victor_left_finger_a_joint_1">
+                <state_interface name="position"/>
+                <state_interface name="effort"/>
             </joint>
         </ros2_control>

Commit message: add finger joints to ros2 control xacro so JS broadcaster will pick up on it

File: victor_moveit_config/config/victor.ros2_control.xacro (robot description, xacro)
@@ -130,4 +130,88 @@
                 <state_interface name="effort"/>
             </joint>
+            <joint name="victor_left_finger_a_joint_2">
+                <state_interface name="position"/>
+                <state_interface name="effort"/>
+            </joint>
+            <joint name="victor_left_finger_a_joint_3">
+                <state_interface name="position"/>
+                <state_interface name="effort"/>
+            </joint>
+            <joint name="victor_left_palm_finger_b_joint">
+                <state_interface name="position"/>
+                <state_interface name="effort"/>
+            </joint>
+            <joint name="victor_left_finger_b_joint_1">
+                <state_interface name="position"/>
+                <state_interface name="effort"/>
+            </joint>
+            <joint name="victor_left_finger_b_joint_2">
+                <state_interface name="position"/>
+                <state_interface name="effort"/>
+            </joint>
+            <joint name="victor_left_finger_b_joint_3">
+                <state_interface name="position"/>
+                <state_interface name="effort"/>
+            </joint>
+            <joint name="victor_left_palm_finger_c_joint">
+                <state_interface name="position"/>
+                <state_interface name="effort"/>
+            </joint>
+            <joint name="victor_left_finger_c_joint_1">
+                <state_interface name="position"/>
+                <state_interface name="effort"/>
+            </joint>
+            <joint name="victor_left_finger_c_joint_2">
+                <state_interface name="position"/>
+                <state_interface name="effort"/>
+            </joint>
+            <joint name="victor_left_finger_c_joint_3">
+                <state_interface name="position"/>
+                <state_interface name="effort"/>
+            </joint>
+            <joint name="victor_right_finger_a_joint_1">
+                <state_interface name="position"/>
+                <state_interface name="effort"/>
+            </joint>
+            <joint name="victor_right_finger_a_joint_2">
+                <state_interface name="position"/>
+                <state_interface name="effort"/>
+            </joint>
+            <joint name="victor_right_finger_a_joint_3">
+                <state_interface name="position"/>
+                <state_interface name="effort"/>
+            </joint>
+            <joint name="victor_right_palm_finger_b_joint">
+                <state_interface name="position"/>
+                <state_interface name="effort"/>
+            </joint>
+            <joint name="victor_right_finger_b_joint_1">
+                <state_interface name="position"/>
+                <state_interface name="effort"/>
+            </joint>
+            <joint name="victor_right_finger_b_joint_2">
+                <state_interface name="position"/>
+                <state_interface name="effort"/>
+            </joint>
+            <joint name="victor_right_finger_b_joint_3">
+                <state_interface name="position"/>
+                <state_interface name="effort"/>
+            </joint>
+            <joint name="victor_right_palm_finger_c_joint">
+                <state_interface name="position"/>
+                <state_interface name="effort"/>
+            </joint>
+            <joint name="victor_right_finger_c_joint_1">
+                <state_interface name="position"/>
+                <state_interface name="effort"/>
+            </joint>
+            <joint name="victor_right_finger_c_joint_2">
+                <state_interface name="position"/>
+                <state_interface name="effort"/>
+            </joint>
+            <joint name="victor_right_finger_c_joint_3">
+                <state_interface name="position"/>
+                <state_interface name="effort"/>
+            </joint>
         </ros2_control>
     </xacro:macro>
