Commit message: victor planning

File: robotiq_3f_description/urdf/robotiq_3f_gripper_macro.xacro (robot description, xacro)
@@ -59,5 +59,5 @@
             <parent link="${prefix}palm"/>
             <child link="${prefix}tool0"/>
-            <origin xyz="0.0 0.0875 0.0" rpy="0 0 1.5707"/>
+            <origin xyz="0.0 0.1475 0.0" rpy="0 0 1.5707"/>
         </joint>
         <!-- end of joint list -->

File: victor_description/urdf/victor.urdf.xacro (robot description, xacro)
@@ -38,13 +38,5 @@
     <link name="$(arg robot_name)_right_arm_world_frame_kuka">
     </link>
-    <!-- arm to gripper adapter -->
-    <xacro:include filename="$(find victor_description)/urdf/iiwa7_to_robotiq_adapter.xacro"/>
-    <xacro:iia7_to_robotiq_adapter parent="$(arg robot_name)_left_arm_flange" prefix="$(arg robot_name)_left">
-        <origin xyz="0 0 -0.01" rpy="0 0 0"/>
-    </xacro:iia7_to_robotiq_adapter>
-    <xacro:iia7_to_robotiq_adapter parent="$(arg robot_name)_right_arm_flange" prefix="$(arg robot_name)_right">
-        <origin xyz="0 0 -0.01" rpy="0 0 0"/>
-    </xacro:iia7_to_robotiq_adapter>
-    <!-- Cartesian commands -->
+        <!-- Cartesian commands -->
     <joint name="$(arg robot_name)_left_arm_cartesian_cmd_joint" type="fixed">
         <origin xyz="0 0 0" rpy="${PI/2} 0 0"/>
@@ -61,4 +53,12 @@
     <link name="$(arg robot_name)_right_arm_cartesian_cmd">
     </link>
+    <!-- arm to gripper adapter -->
+    <xacro:include filename="$(find victor_description)/urdf/iiwa7_to_robotiq_adapter.xacro"/>
+    <xacro:iia7_to_robotiq_adapter parent="$(arg robot_name)_left_arm_flange" prefix="$(arg robot_name)_left">
+        <origin xyz="0 0 -0.01" rpy="0 0 0"/>
+    </xacro:iia7_to_robotiq_adapter>
+    <xacro:iia7_to_robotiq_adapter parent="$(arg robot_name)_right_arm_flange" prefix="$(arg robot_name)_right">
+        <origin xyz="0 0 -0.01" rpy="0 0 0"/>
+    </xacro:iia7_to_robotiq_adapter>
     <!-- Robotiq grippers -->
     <xacro:if value="${gripper == 'robotiq'}">

Commit message: option to disable moveitpy

File: robotiq_3f_description/urdf/robotiq_3f_gripper_macro.xacro (robot description, xacro)
@@ -59,5 +59,5 @@
             <parent link="${prefix}palm"/>
             <child link="${prefix}tool0"/>
-            <origin xyz="0.0 0.1475 0.0" rpy="0 0 1.5707"/>
+            <origin xyz="0.0 0.165 0.0" rpy="0 0 1.5707"/>
         </joint>
         <!-- end of joint list -->

File: victor_description/urdf/iiwa7.xacro (robot description, xacro)
@@ -76,5 +76,5 @@
             <origin xyz="0 0 0.19" rpy="${PI / 2}   0 ${PI}"/>
             <axis xyz="0 0 1"/>
-            <limit lower="${-120 * PI / 180}" upper="${120 * PI / 180}"
+            <limit lower="${-120 * PI / 180}" upper="${119 * PI / 180}"
                    effort="${max_effort}" velocity="1.7453292519943295"/>
             <dynamics damping="${joint_damping}"/>
@@ -226,5 +226,5 @@
             <origin xyz="0 0.081 0.06070" rpy="${- PI / 2} ${PI} 0"/>
             <axis xyz="0 0 1"/>
-            <limit lower="${-175 * PI / 180}" upper="${175 * PI / 180}"
+            <limit lower="${-174 * PI / 180}" upper="${175 * PI / 180}"
                    effort="${max_effort}" velocity="3.141592653589793"/>
             <dynamics damping="${joint_damping}"/>

Commit message: implement circle traj for wrench task

File: robotiq_3f_description/urdf/robotiq_3f_gripper_macro.xacro (robot description, xacro)
@@ -59,5 +59,5 @@
             <parent link="${prefix}palm"/>
             <child link="${prefix}tool0"/>
-            <origin xyz="0.0 0.165 0.0" rpy="0 0 1.5707"/>
+            <origin xyz="0.0 0.1 0.0" rpy="0 0 1.5707"/>
         </joint>
         <!-- end of joint list -->

Commit message: works

File: robotiq_3f_description/urdf/robotiq_3f_gripper_macro.xacro (robot description, xacro)
@@ -59,5 +59,5 @@
             <parent link="${prefix}palm"/>
             <child link="${prefix}tool0"/>
-            <origin xyz="0.0 0.165 0.0" rpy="0 0 1.5707"/>
+            <origin xyz="0.0 0.0 0.0" rpy="0 0 1.5707"/>
         </joint>
         <!-- end of joint list -->

File: victor_description/urdf/victor.urdf (robot description, URDF)
Before this commit: robot victor, 60 links, 59 joints
Joints:
- joint victor_left_palm_tool0: origin xyz=0.0 0.165 0.0 rpy=0 0 1.5707 -> xyz=0.0 0.265 0.0 rpy=0 0 1.5707
- joint victor_right_palm_tool0: origin xyz=0.0 0.165 0.0 rpy=0 0 1.5707 -> xyz=0.0 0.265 0.0 rpy=0 0 1.5707

Commit message: modified teleop logic and button mapping

File: robotiq_3f_description/urdf/robotiq_3f_gripper_macro.xacro (robot description, xacro)
@@ -59,5 +59,5 @@
             <parent link="${prefix}palm"/>
             <child link="${prefix}tool0"/>
-            <origin xyz="0.0 0.0 0.0" rpy="0 0 1.5707"/>
+            <origin xyz="0.0 0.165 0.0" rpy="0 1.5707 1.5707"/>
         </joint>
         <!-- end of joint list -->

File: victor_description/urdf/victor.urdf.xacro (robot description, xacro)
@@ -69,10 +69,10 @@
             <parent link="$(arg robot_name)_left_gripper_mounting_bracket"/>
             <child link="$(arg robot_name)_left_palm"/>
-            <origin xyz="0 0 0.0715" rpy="1.5707 0 0.78539"/>
+            <origin xyz="0 0 0.07" rpy="1.5707963267948966 0 0.7853981633974483"/>
         </joint>
         <joint name="right_gripper_joint" type="fixed">
             <parent link="$(arg robot_name)_right_gripper_mounting_bracket"/>
             <child link="$(arg robot_name)_right_palm"/>
-            <origin xyz="0 0 0.0715" rpy="1.5707 0 0.78539"/>
+            <origin xyz="0 0 0.07" rpy="1.5707 0 0.78539"/>
         </joint>
     </xacro:if>
